File: pcb/pcb-v5/neOSensorV5.sch (KiCad schematic (older format))
At the start: 48 parts, among them J1 Conn_01x04, J2 Conn_01x04, J3 Conn_01x05, J4 Conn_01x05, J5 Conn_01x05, J6 Conn_01x06, Q1 2N7002, SW1 clear, SW2 +, SW3 -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

Commit message: added nodes labels and minor corrections to pcb v5
Parts:
- Q1: footprint Package_TO_SOT_SMD:SOT-23 -> Package_TO_SOT_SMD:SOT-23_Handsoldering
Changed lines of the file:
@@
 F 0 "Q1" H 1530 5454 50  0000 L CNN
 F 1 "2N7002" H 1530 5545 50  0000 L CNN
-F 2 "Package_TO_SOT_SMD:SOT-23" H 1525 5425 50  0001 L CIN
+F 2 "Package_TO_SOT_SMD:SOT-23_Handsoldering" H 1525 5425 50  0001 L CIN
 F 3 "https://www.onsemi.com/pub/Collateral/NDS7002A-D.PDF" H 1325 5500 50  0001 L CNN
 	1    1325 5500

Commit message: update
Connections:
- net +3V3: no longer U3.16 (EN)
- net GND: now also Q1.2 (S); no longer Q1.3 (D)
- net at D1.1 (K): now also Q1.3 (D); no longer Q1.2 (S)
- no-connect marks 12 -> 13
Changed lines of the file:
@@
 encoding utf-8
 Sheet 1 1
-Title "neOSensor v5"
+Title "neOSensor v5.1"
 Date "2021-02-04"
-Rev "v5"
+Rev "v5.1"
 Comp "(c) neOCampus / Dr THIEBOLT François"
-Comment1 "M2siame 2020-2021 project"
-Comment2 "Univ.Tlse3 / IRIT / neOCampus"
+Comment1 "Univ.Tlse3 / IRIT / neOCampus"
+Comment2 "[mar.21][v5.1] corrected Q1 inversion; removed EN tied to 3v3"
 Comment3 ""
 Comment4 ""
@@
 Wire Wire Line
 	8500 5800 8950 5800
-Wire Wire Line
-	8500 2650 8200 2650
-Text Label 8200 2650 0    50   ~ 0
-+3V3
 Text Label 10750 3450 2    50   ~ 0
 TX2
@@
 F 3 "https://www.onsemi.com/pub/Collateral/NDS7002A-D.PDF" H 1325 5500 50  0001 L CNN
 	1    1325 5500
-	-1   0    0    1
+	-1   0    0    -1
 $EndComp
 $Comp
@@
 	0    1    1    0
 $EndComp
+NoConn ~ 8500 2650
 $EndSCHEMATC

Commit message: update neOSensorV5 schematic
Parts:
- removed R6: 470, Resistor_SMD:R_0805_2012Metric_Pad1.20x1.40mm_HandSolder, symbol Device:R_Small
- C2: value 470µF 6.3v -> 100µF 6.3v; footprint Capacitor_THT:CP_Radial_D6.3mm_P2.50mm -> Capacitor_THT:CP_Radial_D5.0mm_P2.50mm
- R1: value 68 -> 150
- R21: value 15K -> 15k
Connections:
- net LED: now also U3.3 (GPIO15); no longer U3.8 (GPIO5)
- net PM_EN: now also U3.8 (GPIO5); no longer U3.4 (GPIO2)
- net RX2: now also U3.6 (GPIO16)
Other:
- note added: "Notes:\n- GPIO5 has a 10k pull-up on +3v3 on devkit V1 !!\n- GPIO5 reserved for Particule Meter ENable (3v3)\n- GPIOX reserved for LED + clear sw\n- GPIO13 reserved for noise sensor\n- GPIO4 reserved for IR sensor (input)\n- ADC2 pins cannot be used when WiFi in use\n- prefer ADC1 pins (GPIO32 --> 39)\n- GPIO1 & GPIO3 are serial0 (prog.)\n- GPIO2 onboard blue led @ devkit V1\n- EN must be floatin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"
- note added: "Red led Vf=1.56v"
- note removed: "Notes:\n- GPIO13 reserved for noise sensor\n- GPIO5 reserved for LED + clear sw\n- GPIO4 reserved for IR sensor\n- ADC2 pins cannot be used when WiFi in use\n- prefer ADC1 pins (GPIO32 --> 39)\n- GPIO1 & GPIO3 are serial0 (prog.)\n- +3V3 on EN pin is optional"
- note removed: "TODO:\n"
Changed lines of the file:
@@
 P 9350 5600
 F 0 "C2" H 9441 5646 50  0000 L CNN
-F 1 "470µF 6.3v" H 9441 5555 50  0000 L CNN
-F 2 "Capacitor_THT:CP_Radial_D6.3mm_P2.50mm" H 9350 5600 50  0001 C CNN
+F 1 "100µF 6.3v" H 9441 5555 50  0000 L CNN
+F 2 "Capacitor_THT:CP_Radial_D5.0mm_P2.50mm" H 9350 5600 50  0001 C CNN
 F 3 "~" H 9350 5600 50  0001 C CNN
 	1    9350 5600
@@
 SDA
 $Comp
-L Device:R_Small R6
-U 1 1 601E5272
-P 9900 3550
-F 0 "R6" V 9900 3550 50  0000 C CNN
-F 1 "470" V 9850 3400 50  0000 C CNN
-F 2 "Resistor_SMD:R_0805_2012Metric_Pad1.20x1.40mm_HandSolder" H 9900 3550 50  0001 C CNN
-F 3 "~" H 9900 3550 50  0001 C CNN
-	1    9900 3550
-	0    1    1    0
-$EndComp
-$Comp
 L Device:R_Small R5
 U 1 1 601E590B
@@
 Wire Wire Line
 	9400 3450 9800 3450
-Wire Wire Line
-	9400 3550 9800 3550
 $Comp
 L power:+3V3 #PWR07
@@
 Power supply
 Text Notes 6050 3100 0    50   ~ 0
-Notes:\n- GPIO13 reserved for noise sensor\n- GPIO5 reserved for LED + clear sw\n- GPIO4 reserved for IR sensor\n- ADC2 pins cannot be used when WiFi in use\n- prefer ADC1 pins (GPIO32 --> 39)\n- GPIO1 & GPIO3 are serial0 (prog.)\n- +3V3 on EN pin is optional
+Notes:\n- GPIO5 has a 10k pull-up on +3v3 on devkit V1 !!\n- GPIO5 reserved for Particule Meter ENable (3v3)\n- GPIOX reserved for LED + clear sw\n- GPIO13 reserved for noise sensor\n- GPIO4 reserved for IR sensor (input)\n- ADC2 pins cannot be used when WiFi in use\n- prefer ADC1 pins (GPIO32 --> 39)\n- GPIO1 & GPIO3 are serial0 (prog.)\n- GPIO2 onboard blue led @ devkit V1\n- EN must be floating !
 $Comp
 L Device:C_Small C1
@@
 NoConn ~ 9400 2850
 NoConn ~ 9400 2950
-Wire Wire Line
-	9700 3750 9400 3750
-Text Label 9700 3750 2    50   ~ 0
-PM_EN
 NoConn ~ 8500 3850
 Wire Wire Line
 	9400 3350 9700 3350
-Text Label 9700 3350 2    50   ~ 0
-LED
-Text Notes 6050 2100 0    50   ~ 0
-TODO:\n
 Text Label 10750 3150 2    50   ~ 0
 INT
@@
 P 1225 4775
 F 0 "R1" V 1225 4775 50  0000 C CNN
-F 1 "68" V 1150 4775 50  0000 C CNN
+F 1 "150" V 1150 4775 50  0000 C CNN
 F 2 "Resistor_SMD:R_0805_2012Metric_Pad1.20x1.40mm_HandSolder" H 1225 4775 50  0001 C CNN
 F 3 "~" H 1225 4775 50  0001 C CNN
@@
 NoConn ~ 8500 3650
 NoConn ~ 8500 3750
-NoConn ~ 9400 3850
 $Comp
 L Amplifier_Operational:LM2902 U5
@@
 P 10175 2550
 F 0 "R21" V 10175 2550 50  0000 C CNN
-F 1 "15K" V 10200 2400 50  0000 C CNN
+F 1 "15k" V 10200 2400 50  0000 C CNN
 F 2 "Resistor_SMD:R_0805_2012Metric_Pad1.20x1.40mm_HandSolder" H 10175 2550 50  0001 C CNN
 F 3 "~" H 10175 2550 50  0001 C CNN
@@
 	1275 7000 1450 7000
 Wire Wire Line
-	10000 3550 10750 3550
-Wire Wire Line
 	10000 3450 10750 3450
 Wire Wire Line
@@
 $EndComp
 NoConn ~ 8500 2650
+Text Label 9700 3350 2    50   ~ 0
+PM_EN
+NoConn ~ 9400 3750
+Wire Wire Line
+	9700 3850 9400 3850
+Text Label 9700 3850 2    50   ~ 0
+LED
+Text Notes 1025 5275 1    50   ~ 0
+Red led Vf=1.56v
+Wire Wire Line
+	9400 3550 10750 3550
 $EndSCHEMATC
