File: pcb/pcb-v5/neOSensorV5.sch (KiCad schematic (older format))
At the start: 47 parts, among them J1 Conn_01x04, J2 Conn_01x04, J3 Conn_01x05, J4 Conn_01x05, J5 Conn_01x05, J6 Conn_01x06, Q1 2N7002, SW1 clear, SW2 +, SW3 -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

Commit message: added note for neOSensor pcb V5.2
Other:
- note added: "- remove R9\n- add 470R in serie withGPIO4 (IR input)"
- note added: ">> TODO: neOSensor V5.2 <<"
- note removed: "TODO:\n- remove R9\n- add 470R in serie withGPIO4 (IR input)"
Changed lines of the file:
@@
 Wire Wire Line
 	9400 3550 10750 3550
-Text Notes 5000 3575 0    50   ~ 0
-TODO:\n- remove R9\n- add 470R in serie withGPIO4 (IR input)
+Text Notes 5000 3600 0    50   ~ 0
+- remove R9\n- add 470R in serie withGPIO4 (IR input)
 Wire Notes Line
 	4975 3275 6850 3275
@@
 Wire Notes Line
 	4950 4025 4950 3275
+Text Notes 5000 3425 0    71   ~ 14
+>> TODO: neOSensor V5.2 <<
 $EndSCHEMATC
