File: pcb/pcb-v5/neOSensorV5.kicad_pcb (KiCad board)
At the start: 2 copper layers, 49.5 x 49.5 mm, 47 parts, among them J1 Conn_01x04, J2 Conn_01x04, J3 Conn_01x05, J4 Conn_01x05, J5 Conn_01x05, J6 Conn_01x06, Q1 2N7002, SW1 clear, SW2 +, SW3 -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

Commit message: new neOSensor V5.1 PCB done :)
Parts:
- added REF**: KiCad-Logo_8mm_SilkScreen, Symbol:KiCad-Logo_8mm_SilkScreen, B.Cu at (44.5, 59.1)
- added REF**: WEEE-Logo_4.2x6mm_SilkScreen, Symbol:WEEE-Logo_4.2x6mm_SilkScreen, B.Cu at (66.3, 44.6)
- added REF**: ESD-Logo_6.6x6mm_SilkScreen, Symbol:ESD-Logo_6.6x6mm_SilkScreen, F.Cu at (42.5, 60.3)
- added REF**: RoHS-Logo_6mm_SilkScreen, Symbol:RoHS-Logo_6mm_SilkScreen, F.Cu at (58.0, 60.3)
- added REF**: CE-Logo_8.5x6mm_SilkScreen, Symbol:CE-Logo_8.5x6mm_SilkScreen, F.Cu at (34.2, 34.2)
- added REF**: OSHW-Logo_7.5x8mm_SilkScreen, Symbol:OSHW-Logo_7.5x8mm_SilkScreen, F.Cu at (63.9, 70.5)
Other:
- board text added: "M2SIAME apr.21"
- board text added: "Sensor v5.1"
- board text added: "Univ-Tlse3/IRIT"
- board text removed: "M2SIAME FEB21 FE/FT"
- board text removed: "Sensor v5"
- board text removed: "Univ.Tlse3/IRIT"
