File: pcb/pcb-v5/neOSensorv5_panelized.kicad_pcb (KiCad board)
At the start: 2 copper layers, 99.9 x 99.9 mm, 196 parts, among them J1 Conn_01x04, J2 Conn_01x04, J3 Conn_01x05, J4 Conn_01x05, J5 Conn_01x05, J6 Conn_01x06, Q1 2N7002, SW1 clear, SW2 +, SW3 -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

Commit message: new neOSensor V5.1 PCB done :)
Parts:
- removed the C2 at (39.9, 69.3)
- removed the C2 at (90.3, 69.3)
- removed the C2 at (60.5, 81.4)
- removed the C2 at (110.9, 81.4)
- removed the Q1 at (36.7, 33.7)
- removed the Q1 at (87.1, 33.7)
- removed the Q1 at (63.6, 117.1)
- removed the Q1 at (114.0, 117.1)
- removed R6 (x4): 470, Resistor_SMD:R_0805_2012Metric_Pad1.20x1.40mm_HandSolder
- removed the REF** at (63.6, 70.4)
- removed the REF** at (114.0, 70.4)
- removed the REF** at (36.7, 80.4)
- removed the REF** at (87.1, 80.4)
- added C2: 100µF 6.3v, Capacitor_THT:CP_Radial_D5.0mm_P2.50mm, F.Cu at (60.5, 81.4)
- added C2: 100µF 6.3v, Capacitor_THT:CP_Radial_D5.0mm_P2.50mm, F.Cu at (110.9, 81.4)
- added C2: 100µF 6.3v, Capacitor_THT:CP_Radial_D5.0mm_P2.50mm, F.Cu at (90.3, 69.3)
- added C2: 100µF 6.3v, Capacitor_THT:CP_Radial_D5.0mm_P2.50mm, F.Cu at (39.9, 69.3)
- added Q1: 2N7002, Package_TO_SOT_SMD:SOT-23_Handsoldering, B.Cu at (63.9, 118.5)
- added Q1: 2N7002, Package_TO_SOT_SMD:SOT-23_Handsoldering, B.Cu at (114.4, 118.5)
- added Q1: 2N7002, Package_TO_SOT_SMD:SOT-23_Handsoldering, B.Cu at (86.8, 32.3)
- added Q1: 2N7002, Package_TO_SOT_SMD:SOT-23_Handsoldering, B.Cu at (36.4, 32.3)
- added REF**: WEEE-Logo_4.2x6mm_SilkScreen, Symbol:WEEE-Logo_4.2x6mm_SilkScreen, B.Cu at (34.0, 106.2)
- added REF**: RoHS-Logo_6mm_SilkScreen, Symbol:RoHS-Logo_6mm_SilkScreen, F.Cu at (92.7, 90.4)
- added REF**: CE-Logo_8.5x6mm_SilkScreen, Symbol:CE-Logo_8.5x6mm_SilkScreen, F.Cu at (116.6, 116.6)
- added REF**: ESD-Logo_6.6x6mm_SilkScreen, Symbol:ESD-Logo_6.6x6mm_SilkScreen, F.Cu at (108.2, 90.4)
- added REF**: WEEE-Logo_4.2x6mm_SilkScreen, Symbol:WEEE-Logo_4.2x6mm_SilkScreen, B.Cu at (116.7, 44.6)
- added REF**: KiCad-Logo_8mm_SilkScreen, Symbol:KiCad-Logo_8mm_SilkScreen, B.Cu at (94.9, 59.1)
- added REF**: ESD-Logo_6.6x6mm_SilkScreen, Symbol:ESD-Logo_6.6x6mm_SilkScreen, F.Cu at (93.0, 60.3)
- added REF**: OSHW-Logo_7.5x8mm_SilkScreen, Symbol:OSHW-Logo_7.5x8mm_SilkScreen, F.Cu at (114.3, 70.5)
- added REF**: CE-Logo_8.5x6mm_SilkScreen, Symbol:CE-Logo_8.5x6mm_SilkScreen, F.Cu at (84.6, 34.2)
- added REF**: RoHS-Logo_6mm_SilkScreen, Symbol:RoHS-Logo_6mm_SilkScreen, F.Cu at (108.5, 60.3)
- added REF**: KiCad-Logo_8mm_SilkScreen, Symbol:KiCad-Logo_8mm_SilkScreen, B.Cu at (44.5, 59.1)
- added REF**: KiCad-Logo_8mm_SilkScreen, Symbol:KiCad-Logo_8mm_SilkScreen, B.Cu at (55.9, 91.7)
- added REF**: WEEE-Logo_4.2x6mm_SilkScreen, Symbol:WEEE-Logo_4.2x6mm_SilkScreen, B.Cu at (66.3, 44.6)
- added REF**: ESD-Logo_6.6x6mm_SilkScreen, Symbol:ESD-Logo_6.6x6mm_SilkScreen, F.Cu at (42.5, 60.3)
- added REF**: RoHS-Logo_6mm_SilkScreen, Symbol:RoHS-Logo_6mm_SilkScreen, F.Cu at (58.0, 60.3)
- added REF**: CE-Logo_8.5x6mm_SilkScreen, Symbol:CE-Logo_8.5x6mm_SilkScreen, F.Cu at (34.2, 34.2)
- added REF**: OSHW-Logo_7.5x8mm_SilkScreen, Symbol:OSHW-Logo_7.5x8mm_SilkScreen, F.Cu at (63.9, 70.5)
- added REF**: RoHS-Logo_6mm_SilkScreen, Symbol:RoHS-Logo_6mm_SilkScreen, F.Cu at (42.3, 90.4)
- added REF**: CE-Logo_8.5x6mm_SilkScreen, Symbol:CE-Logo_8.5x6mm_SilkScreen, F.Cu at (66.2, 116.6)
- added REF**: OSHW-Logo_7.5x8mm_SilkScreen, Symbol:OSHW-Logo_7.5x8mm_SilkScreen, F.Cu at (36.4, 80.3)
- added REF**: ESD-Logo_6.6x6mm_SilkScreen, Symbol:ESD-Logo_6.6x6mm_SilkScreen, F.Cu at (57.8, 90.4)
- added REF**: KiCad-Logo_8mm_SilkScreen, Symbol:KiCad-Logo_8mm_SilkScreen, B.Cu at (106.3, 91.7)
- added REF**: WEEE-Logo_4.2x6mm_SilkScreen, Symbol:WEEE-Logo_4.2x6mm_SilkScreen, B.Cu at (84.5, 106.2)
- added REF**: OSHW-Logo_7.5x8mm_SilkScreen, Symbol:OSHW-Logo_7.5x8mm_SilkScreen, F.Cu at (86.9, 80.3)
- R1 (x4): value 68 -> 150
- R21 (x4): value 15K -> 15k
Connections:
- U3 pad 16: +3V3 -> Net-(U3-Pad16) (x4)
- U3 pad 3: Net-(U3-Pad3) -> /LED (x4)
- U3 pad 4: /PM_EN -> Net-(U3-Pad4) (x4)
- U3 pad 6: Net-(R6-Pad2) -> /RX2 (x4)
- U3 pad 8: /LED -> /PM_EN (x4)
Routing:
- net +3V3: track 756.5 -> 631.8 mm, vias 100 -> 92
- net /RX2: track 11.8 -> 136.3 mm, vias 0 -> 12
- net Net-(R6-Pad2): track 116.6 -> 0.00 mm, vias 12 -> 0
- net /LED: track 79.6 -> 29.9 mm, vias 12 -> 0
- net /PM_EN: track 144.6 -> 102.8 mm
- net Net-(D1-Pad1): track 17.9 -> 11.5 mm, vias 0 -> 4
- net Net-(Q1-Pad1): track 27.7 -> 33.7 mm
- net /SCL: track 545.7 -> 546.4 mm
Other:
- board text added: "IR"
- board text added: "M2SIAME apr.21"
- board text added: "Sensor v5.1"
- board text added: "Univ-Tlse3/IRIT"
- board text removed: "M2SIAME FEB21 FE/FT"
- board text removed: "Sensor v5"
- board text removed: "Univ.Tlse3/IRIT"
