File: pcb/lorawan/neOSensor Cubecell_V1.kicad_pcb (KiCad board)
At the start: 2 copper layers, 47 x 44.5 mm, 20 parts, among them J1 Conn_01x05, J2 Conn_01x05, J3 Conn_01x04, J4 Conn_01x04, J5 Conn_01x05, J6 Conn_01x04, SW1 G71Y, U1 HTCC-AB01

Commit message: update
Parts:
- added J7: 78_01_030_0004, neosensor_addon:ATECC508A, F.Cu at (210.1, 86.4)
Routing:
- net /GND: track 14.3 -> 24.8 mm
- net /SCL: track 110.3 -> 115.9 mm
- net /Vsensor: track 89.2 -> 92.2 mm
- net /SDA: track 105.5 -> 107.2 mm
Changed lines of the file:
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@@
     (thickness 1.6)
     (drawings 44)
-    (tracks 153)
+    (tracks 166)
     (zones 0)
-    (modules 20)
-    (nets 22)
+    (modules 21)
+    (nets 26)
   )
   (page A4)
@@
     (34 B.Paste user)
     (35 F.Paste user)
-    (36 B.SilkS user)
+    (36 B.SilkS user hide)
     (37 F.SilkS user)
     (38 B.Mask user)
@@
   (net 20 /RST)
   (net 21 /Vsensor)
+  (net 22 "Net-(J7-Pad7)")
+  (net 23 "Net-(J7-Pad3)")
+  (net 24 "Net-(J7-Pad2)")
+  (net 25 "Net-(J7-Pad1)")
   (net_class Default "This is the default net class."
     (clearance 0.1524)
@@
     (add_net /SDA)
     (add_net /TX)
+    (add_net "Net-(J7-Pad1)")
+    (add_net "Net-(J7-Pad2)")
+    (add_net "Net-(J7-Pad3)")
+    (add_net "Net-(J7-Pad7)")
   )
   (net_class Power ""
@@
     (add_net /VS*)
     (add_net /Vsensor)
+  )
+  (module neosensor_addon:ATECC508A (layer F.Cu)
+    (at 210.058 86.36 180)
+    (fp_text reference J7 (at -0.535 -3.342) (layer F.SilkS)
+      (effects (font (size 1 1) (thickness 0.015)))
+    )
+    (fp_text value 78_01_030_0004 (at 7.72 3.342) (layer F.Fab)
+      (effects (font (size 1 1) (thickness 0.015)))
+    )
+    (fp_line (start 3.71 -2.75) (end 3.71 2.75) (layer F.CrtYd) (width 0.05))
+    (fp_line (start -3.71 -2.75) (end -3.71 2.75) (layer F.CrtYd) (width 0.05))
+    (fp_line (start -3.71 2.75) (end 3.71 2.75) (layer F.CrtYd) (width 0.05))
+    (fp_line (start -3.71 -2.75) (end 3.71 -2.75) (layer F.CrtYd) (width 0.05))
+    (fp_line (start 2 -2.5) (end 2 2.5) (layer F.Fab) (width 0.127))
+    (fp_line (start -2 -2.5) (end -2 2.5) (layer F.Fab) (width 0.127))
+    (fp_line (start -2 2.53) (end 2 2.53) (layer F.SilkS) (width 0.127))
+    (fp_line (start -2 -2.53) (end 2 -2.53) (layer F.SilkS) (width 0.127))
+    (fp_line (start -2 2.5) (end 2 2.5) (layer F.Fab) (width 0.127))
+    (fp_line (start -2 -2.5) (end 2 -2.5) (layer F.Fab) (width 0.127))
+    (fp_circle (center -4.315 -2.515) (end -4.215 -2.515) (layer F.Fab) (width 0.2))
+    (fp_circle (center -4.315 -2.515) (end -4.215 -2.515) (layer F.SilkS) (width 0.2))
+    (pad 8 smd rect (at 2.605 -1.905 180) (size 1.71 0.61) (layers F.Cu F.Paste F.Mask)
+      (net 21 /Vsensor))
+    (pad 7 smd rect (at 2.605 -0.635 180) (size 1.71 0.61) (layers F.Cu F.Paste F.Mask)
+      (net 22 "Net-(J7-Pad7)"))
+    (pad 6 smd rect (at 2.605 0.635 180) (size 1.71 0.61) (layers F.Cu F.Paste F.Mask)
+      (net 16 /SCL))
+    (pad 5 smd rect (at 2.605 1.905 180) (size 1.71 0.61) (layers F.Cu F.Paste F.Mask)
+      (net 15 /SDA))
+    (pad 4 smd rect (at -2.605 1.905 180) (size 1.71 0.61) (layers F.Cu F.Paste F.Mask)
+      (net 11 /GND))
+    (pad 3 smd rect (at -2.605 0.635 180) (size 1.71 0.61) (layers F.Cu F.Paste F.Mask)
+      (net 23 "Net-(J7-Pad3)"))
+    (pad 2 smd rect (at -2.605 -0.635 180) (size 1.71 0.61) (layers F.Cu F.Paste F.Mask)
+      (net 24 "Net-(J7-Pad2)"))
+    (pad 1 smd rect (at -2.605 -1.905 180) (size 1.71 0.61) (layers F.Cu F.Paste F.Mask)
+      (net 25 "Net-(J7-Pad1)"))
   )
   (module Symbol:OSHW-Logo2_9.8x8mm_SilkScreen (layer B.Cu)
@@
   (segment (start 219.075 94.488) (end 219.075 91.678318) (width 0.6604) (layer B.Cu) (net 11))
   (segment (start 223.796399 90.700399) (end 225.298 92.202) (width 0.6604) (layer B.Cu) (net 11))
+  (segment (start 211.904318 84.455) (end 211.325399 85.033919) (width 0.6604) (layer F.Cu) (net 11))
+  (segment (start 211.325399 85.033919) (end 211.325399 89.659399) (width 0.6604) (layer F.Cu) (net 11))
+  (segment (start 212.663 84.455) (end 211.904318 84.455) (width 0.6604) (layer F.Cu) (net 11))
+  (segment (start 210.814798 90.17) (end 207.155 90.17) (width 0.6604) (layer F.Cu) (net 11))
+  (segment (start 211.325399 89.659399) (end 210.814798 90.17) (width 0.6604) (layer F.Cu) (net 11))
   (via (at 223.52 66.04) (size 1.2) (drill 0.6) (layers F.Cu B.Cu) (net 12))
   (segment (start 226.568 66.04) (end 223.52 66.04) (width 0.6604) (layer B.Cu) (net 12))
@@
   (segment (start 213.4806 55.2514) (end 213.4806 73.66) (width 0.2032) (layer F.Cu) (net 15))
   (segment (start 213.4806 54.154681) (end 213.4806 55.2514) (width 0.2032) (layer F.Cu) (net 15))
+  (segment (start 207.01 84.012) (end 207.453 84.455) (width 0.2032) (layer F.Cu) (net 15))
+  (segment (start 207.01 82.931) (end 207.01 84.012) (width 0.2032) (layer F.Cu) (net 15))
   (segment (start 196.85 93.218) (end 196.85 86.995) (width 0.2032) (layer F.Cu) (net 16))
   (segment (start 196.85 86.995) (end 196.342 86.487) (width 0.2032) (layer F.Cu) (net 16))
@@
   (segment (start 210.82 55.88) (end 210.82 71.12) (width 0.2032) (layer F.Cu) (net 16))
   (segment (start 210.82 52.832) (end 210.82 55.88) (width 0.2032) (layer F.Cu) (net 16))
+  (segment (start 204.47 82.607685) (end 204.47 82.042) (width 0.2032) (layer F.Cu) (net 16))
+  (segment (start 204.47 83.8002) (end 204.47 82.607685) (width 0.2032) (layer F.Cu) (net 16))
+  (segment (start 206.3948 85.725) (end 204.47 83.8002) (width 0.2032) (layer F.Cu) (net 16))
+  (segment (start 207.453 85.725) (end 206.3948 85.725) (width 0.2032) (layer F.Cu) (net 16))
   (via (at 220.98 91.694) (size 0.8) (drill 0.4) (layers F.Cu B.Cu) (net 19))
   (segment (start 221.039 91.753) (end 220.98 91.694) (width 0.2032) (layer B.Cu) (net 19))
@@
   (via (at 187.96 83.312) (size 1.2) (drill 0.6) (layers F.Cu B.Cu) (net 21))
   (segment (start 187.96 83.312) (end 187.96 68.58) (width 0.6604) (layer F.Cu) (net 21))
+  (segment (start 206.883 88.265) (end 207.453 88.265) (width 0.6604) (layer F.Cu) (net 21))
+  (segment (start 205.105 90.043) (end 206.883 88.265) (width 0.6604) (layer F.Cu) (net 21))
   (zone (net 11) (net_name /GND) (layer F.Cu) (hatch edge 0.508)
     (connect_pads (clearance 0.254))

Commit message: update
Parts:
- removed C2, C4: 100n, Capacitor_SMD:C_0805_2012Metric_Pad1.15x1.40mm_HandSolder
- removed J4: Conn_01x04, Connector_PinHeader_2.54mm:PinHeader_1x04_P2.54mm_Vertical
- added U2: HC-SR01, neosensor_addon:PIR_HC-SR01, B.Cu at (72.7, 57.6)
- added U3: OLED1.3_I2C, neosensor_addon:OLED1.3_I2C, B.Cu at (74.0, 55.8)
- J7: value 78_01_030_0004 -> ATECC508A
- moved J7 147.9 mm to (63.1, 69.6), turned to 0 degrees
- moved R1 137.4 mm to (77.2, 61.2)
- moved R2 137.4 mm to (77.2, 46.4)
- moved U1 137.4 mm to (65.6, 53.6)
- moved MH2 137.2 mm to (48.7, 78.1)
- moved J5 136.4 mm to (50.5, 33.4)
- moved J1 136.3 mm to (70.8, 33.4)
- moved C3 136.0 mm to (71.2, 73.3)
- moved JP1 136.0 mm to (53.0, 51.7)
- moved C1 136.0 mm to (71.8, 39.0)
- moved C5 136.0 mm to (51.5, 39.0)
- moved C6 135.7 mm to (57.8, 75.6)
- moved SW1 135.7 mm to (88.3, 81.3)
- moved J6 135.6 mm to (56.8, 79.7)
- moved J3 135.6 mm to (70.2, 79.7)
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Connections:
- JP1 pad 1: /VEXT -> /VDD
- JP1 pad 3: /VDD -> /VEXT
Routing:
- net /SDA: track 107.2 -> 128.3 mm, vias 8 -> 11
- net /Vsensor: track 92.2 -> 107.6 mm, vias 10 -> 8
- net /SCL: track 115.9 -> 130.3 mm, vias 8 -> 10
- net /GPIO1: track 57.9 -> 66.4 mm
- net /GND: track 24.8 -> 16.7 mm
- net /GPIO0: track 0.00 -> 4.17 mm
- net /GPIO5: track 17.1 -> 20.7 mm
- net /VEXT: track 22.0 -> 23.2 mm
- net /VIN: track 36.1 -> 35.2 mm
- net /VDD: track 64.4 -> 63.8 mm
Other:
- board size 47 x 44.5 mm -> 50 x 50 mm
- board text added: "05/2021"
- board text removed: "JM 09/2020"

Commit message: mise a jour des schema
Parts:
- removed J7: ATECC508A, neosensor_addon:ATECC508A
- added U5: ATECC508A, neosensor_addon:SOIC-8_3.9x5.4mm_P1.27mm_HandSolder, F.Cu at (63.2, 69.6)
- SW1: moved to F.Cu
- U1: footprint HTCC-AB01:htcc-ab01 -> neosensor_addon:HTCC-AB01
- moved SW1 0.26 mm to (88.1, 81.4), turned to 180 degrees
- moved U1 0.18 mm to (65.6, 53.4)
Routing:
- net /GND: track 16.7 -> 13.2 mm
- net /GPIO5: track 20.7 -> 22.4 mm, vias 2 -> 3

Commit message: update
Parts:
- removed C5, C6: 100n, Capacitor_SMD:C_0805_2012Metric_Pad1.15x1.40mm_HandSolder
- added C2: 100nF, Capacitor_SMD:C_0805_2012Metric_Pad1.15x1.40mm_HandSolder, B.Cu at (56.9, 46.5)
- added IR1: IRsensor, neosensor_addon:IRsensor_TH_and_smd, F.Cu at (63.0, 51.6)
- added R4: 15K, Resistor_SMD:R_0805_2012Metric_Pad1.15x1.40mm_HandSolder, F.Cu at (89.3, 76.0)
- added R5: 15K, Resistor_SMD:R_0805_2012Metric_Pad1.15x1.40mm_HandSolder, F.Cu at (90.3, 72.5)
- added U4: AMS1117, Package_TO_SOT_SMD:SOT-223-3_TabPin2, B.Cu at (49.1, 69.5)
- C1: value 100n -> 1µF; footprint Capacitor_SMD:C_0805_2012Metric_Pad1.15x1.40mm_HandSolder -> Resistor_SMD:R_0805_2012Metric_Pad1.20x1.40mm_HandSolder
- C3: value 100n -> 100µF; footprint Capacitor_SMD:C_0805_2012Metric_Pad1.15x1.40mm_HandSolder -> Capacitor_THT:CP_Radial_D5.0mm_P2.50mm; moved to B.Cu
- JP1: moved to F.Cu
- moved C1 36.7 mm to (86.9, 72.5), turned to 270 degrees
- moved C3 27.6 mm to (49.5, 56.2), turned to 180 degrees
- moved JP1 0.19 mm to (53.0, 51.9), turned to 0 degrees
- moved MH1 0.11 mm to (91.8, 35.0)
Connections:
- net /GPIO0 renamed /IR
- C1 pad 1: /Vsensor -> /GPIO5
- C3 pad 1: /Vsensor -> /3v3
- J2 pad 1: /VDD -> /Vsensor
- JP1 pad 1: /VDD -> /3v3
- JP1 pad 3: /VEXT -> /VDD
- R1 pad 2: /VIN -> /Vsensor
- R2 pad 2: /VIN -> /Vsensor
- SW1 pad 1: /GPIO5 -> Net-(R4-Pad1)
- SW1 pad 2: /GND -> /Vsensor
Routing:
- net /Vsensor: track 107.6 -> 186.4 mm, vias 8 -> 17
- net /VDD: track 63.8 -> 18.3 mm, vias 5 -> 3
- net /VEXT: track 23.2 -> 0.02 mm, vias 3 -> 0
- net /3v3: track 0.00 -> 23.2 mm, vias 0 -> 4
- net /IR: track 4.17 -> 25.1 mm, vias 0 -> 2
- net /GND: track 13.2 -> 0.00 mm, vias 16 -> 19
- net /VIN: track 35.2 -> 40.8 mm, vias 3 -> 6
- net Net-(R4-Pad1): track 0.00 -> 5.21 mm
- net /GPIO5: track 22.4 -> 22.3 mm, vias 3 -> 5

Commit message: update
Parts:
- IR1: moved to B.Cu
- moved U2 7.76 mm to (69.5, 50.5)
- moved U3 0.37 mm to (74.0, 55.5)
- turned IR1 to 0 degrees
Connections:
- U2 pad 1: /Vsensor -> /VIN
Routing:
- net /VIN: track 40.8 -> 49.7 mm
- net /IR: track 25.1 -> 22.1 mm, vias 2 -> 3
- net /Vsensor: track 186.4 -> 187.7 mm, vias 17 -> 18
