File: pcb/lorawan/neOSensor Cubecell_V1.sch (KiCad schematic (older format))
At the start: 19 parts, among them J1 Conn_01x05, J2 Conn_01x05, J3 Conn_01x04, J4 Conn_01x04, J5 Conn_01x05, J6 Conn_01x04, SW1 G71Y, U1 HTCC-AB01

Commit message: update
Parts:
- added J7: 78_01_030_0004, neosensor_addon:ATECC508A, symbol ATECC508A:78_01_030_0004
- SW1: symbol neosensor_addon:G71Y -> neOSensor_Cubecell_V1-rescue:G71Y-neosensor_addon
- U1: symbol htcc-ab01:HTCC-AB01 -> neOSensor_Cubecell_V1-rescue:HTCC-AB01-htcc-ab01
Connections:
- no-connect marks 0 -> 4
Other:
- note added: "ATECC508A-SSHDA"
Changed lines of the file:
@@
 $EndDescr
 $Comp
-L htcc-ab01:HTCC-AB01 U1
+L neOSensor_Cubecell_V1-rescue:HTCC-AB01-htcc-ab01 U1
 U 1 1 5F579B0C
 P 4900 3100
@@
 Expansion connectors for screen\n\n\n
 $Comp
-L neosensor_addon:G71Y SW1
+L neOSensor_Cubecell_V1-rescue:G71Y-neosensor_addon SW1
 U 1 1 5F5ADA5E
 P 10000 4400
@@
 	1    0    0    -1
 $EndComp
+Text Notes 9345 5915 0    50   ~ 0
+ATECC508A-SSHDA
+Wire Notes Line
+	9115 5995 9115 5035
+Text Label 10085 5570 0    50   ~ 0
+SCL
+Text Label 10085 5670 0    50   ~ 0
+SDA
+Text Label 9285 5670 2    50   ~ 0
+GND
+Text Label 10085 5370 0    50   ~ 0
+Vsensor
+Wire Notes Line
+	10395 5035 10395 5995
+Wire Notes Line
+	9115 5035 10395 5035
+Wire Notes Line
+	9115 5995 10395 5995
+NoConn ~ 10085 5470
+NoConn ~ 9285 5370
+NoConn ~ 9285 5470
+NoConn ~ 9285 5570
+$Comp
+L ATECC508A:78_01_030_0004 J7
+U 1 1 60AE7AA0
+P 9685 5470
+F 0 "J7" H 9685 5837 50  0000 C CNN
+F 1 "78_01_030_0004" H 9685 5746 50  0000 C CNN
+F 2 "neosensor_addon:ATECC508A" H 9685 5470 50  0001 L BNN
+F 3 "" H 9685 5470 50  0001 L BNN
+F 4 "Harting" H 9685 5470 50  0001 L BNN "MANUFACTURER"
+F 5 "2021-04-27" H 9685 5470 50  0001 L BNN "PARTREV"
+F 6 "8 mm" H 9685 5470 50  0001 L BNN "MAXIMUM_PACKAGE_HEIGHT"
+F 7 "Manufacturer Recommendations" H 9685 5470 50  0001 L BNN "STANDARD"
+	1    9685 5470
+	1    0    0    -1
+$EndComp

Commit message: update
Parts:
- removed C2, C4: 100n, Capacitor_SMD:C_0805_2012Metric_Pad1.15x1.40mm_HandSolder, symbol Device:C_Small
- removed J4: Conn_01x04, Connector_PinHeader_2.54mm:PinHeader_1x04_P2.54mm_Vertical, symbol Connector_Generic:Conn_01x04
- removed J7: 78_01_030_0004, neosensor_addon:ATECC508A, symbol ATECC508A:78_01_030_0004
- added C?: 100nF, symbol Device:C
- added C?: C, symbol Device:C
- added J7: ATECC508A, neosensor_addon:ATECC508A, symbol neosensor_addon:ATECC508A
- added U2: HC-SR01, neosensor_addon:PIR_HC-SR01, symbol neosensor_addon:HC-SR01
- added U3: OLED1.3_I2C, neosensor_addon:OLED1.3_I2C, symbol neosensor_addon:OLED1.3_I2C
- added U?: AMS1117, Package_TO_SOT_SMD:SOT-223-3_TabPin2, symbol Regulator_Linear:AMS1117
- SW1: symbol neOSensor_Cubecell_V1-rescue:G71Y-neosensor_addon -> neOSensor-Cubecell_V1-rescue:G71Y-neosensor_addon-neOSensor_Cubecell_V1-rescue
- U1: symbol neOSensor_Cubecell_V1-rescue:HTCC-AB01-htcc-ab01 -> neOSensor-Cubecell_V1-rescue:HTCC-AB01-htcc-ab01-neOSensor_Cubecell_V1-rescue
Connections:
- wire segments 84 -> 83
Other:
- note removed: "Expansion connectors for screen\n\n\n"
Changed lines of the file:
@@
 $EndDescr
 $Comp
-L neOSensor_Cubecell_V1-rescue:HTCC-AB01-htcc-ab01 U1
+L neOSensor-Cubecell_V1-rescue:HTCC-AB01-htcc-ab01-neOSensor_Cubecell_V1-rescue U1
 U 1 1 5F579B0C
 P 4900 3100
@@
 Wire Wire Line
 	9100 2500 8900 2500
-Text Label 8600 2400 3    50   ~ 0
-VDD
 Text Label 8800 2400 3    50   ~ 0
 GND
@@
 Vsensor
 $Comp
-L Connector_Generic:Conn_01x04 J4
-U 1 1 5F591203
-P 10100 3200
-F 0 "J4" H 10180 3192 50  0000 L CNN
-F 1 "Conn_01x04" H 10180 3101 50  0000 L CNN
-F 2 "Connector_PinHeader_2.54mm:PinHeader_1x04_P2.54mm_Vertical" H 10100 3200 50  0001 C CNN
-F 3 "~" H 10100 3200 50  0001 C CNN
-	1    10100 3200
-	1    0    0    -1
-$EndComp
-Wire Wire Line
-	9900 3300 9700 3300
-Wire Wire Line
-	9900 3400 9700 3400
-Text Label 9200 3400 3    50   ~ 0
-GND
-Text Label 9400 3400 3    50   ~ 0
-Vsensor
-Text Label 9700 3300 0    50   ~ 0
-SCL
-Text Label 9700 3400 0    50   ~ 0
-SDA
-Text Notes 9500 3000 0    50   ~ 0
-Expansion connectors for screen\n\n\n
-$Comp
-L neOSensor_Cubecell_V1-rescue:G71Y-neosensor_addon SW1
+L neOSensor-Cubecell_V1-rescue:G71Y-neosensor_addon-neOSensor_Cubecell_V1-rescue SW1
 U 1 1 5F5ADA5E
 P 10000 4400
@@
 Text Label 9400 1300 0    50   ~ 0
 Vsensor
+Text Label 9900 1700 0    50   ~ 0
+VEXT
+Wire Wire Line
+	9900 1500 9900 1700
 Text Label 9900 1000 0    50   ~ 0
-VEXT
-Wire Wire Line
-	9900 1500 9900 1700
-Text Label 9900 1700 0    50   ~ 0
 VDD
-$Comp
-L Device:C_Small C2
-U 1 1 5F593B1B
-P 8700 2200
-F 0 "C2" V 8929 2200 50  0000 C CNN
-F 1 "100n" V 8838 2200 50  0000 C CNN
-F 2 "Capacitor_SMD:C_0805_2012Metric_Pad1.15x1.40mm_HandSolder" H 8700 2200 50  0001 C CNN
-F 3 "~" H 8700 2200 50  0001 C CNN
-	1    8700 2200
-	0    -1   -1   0
-$EndComp
-$Comp
-L Device:C_Small C4
-U 1 1 5F595F37
-P 9300 3200
-F 0 "C4" V 9529 3200 50  0000 C CNN
-F 1 "100n" V 9438 3200 50  0000 C CNN
-F 2 "Capacitor_SMD:C_0805_2012Metric_Pad1.15x1.40mm_HandSolder" H 9300 3200 50  0001 C CNN
-F 3 "~" H 9300 3200 50  0001 C CNN
-	1    9300 3200
-	0    -1   -1   0
-$EndComp
-Wire Wire Line
-	8600 2100 8600 2200
-Connection ~ 8600 2200
-Wire Wire Line
-	8600 2200 8600 2400
 Wire Wire Line
 	8600 2100 9100 2100
@@
 Wire Wire Line
 	8800 2200 8800 2400
-Connection ~ 8800 2200
 Wire Wire Line
 	7200 2100 7800 2100
@@
 Text Label 6100 2800 0    50   ~ 0
 GPIO2
-Wire Wire Line
-	9200 3100 9200 3200
-Wire Wire Line
-	9200 3100 9900 3100
-Connection ~ 9200 3200
-Wire Wire Line
-	9200 3200 9200 3400
-Wire Wire Line
-	9400 3200 9900 3200
-Wire Wire Line
-	9400 3200 9400 3400
-Connection ~ 9400 3200
 $Comp
 L Mechanical:MountingHole_Pad MH1
@@
 Text Notes 9345 5915 0    50   ~ 0
 ATECC508A-SSHDA
-Wire Notes Line
-	9115 5995 9115 5035
 Text Label 10085 5570 0    50   ~ 0
 SCL
@@
 Text Label 10085 5370 0    50   ~ 0
 Vsensor
-Wire Notes Line
-	10395 5035 10395 5995
-Wire Notes Line
-	9115 5035 10395 5035
-Wire Notes Line
-	9115 5995 10395 5995
 NoConn ~ 10085 5470
 NoConn ~ 9285 5370
@@
 NoConn ~ 9285 5570
 $Comp
-L ATECC508A:78_01_030_0004 J7
-U 1 1 60AE7AA0
+L neosensor_addon:HC-SR01 U2
+U 1 1 60B0C27A
+P 6840 5635
+F 0 "U2" H 7168 5739 50  0000 L CNN
+F 1 "HC-SR01" H 7168 5648 50  0000 L CNN
+F 2 "neosensor_addon:PIR_HC-SR01" H 6840 5635 50  0001 C CNN
+F 3 "" H 6840 5635 50  0001 C CNN
+	1    6840 5635
+	1    0    0    -1
+$EndComp
+$Comp
+L neosensor_addon:OLED1.3_I2C U3
+U 1 1 60B0C862
+P 8455 5800
+F 0 "U3" H 8933 5804 50  0000 L CNN
+F 1 "OLED1.3_I2C" H 8933 5713 50  0000 L CNN
+F 2 "neosensor_addon:OLED1.3_I2C" H 8455 5800 50  0001 C CNN
+F 3 "" H 8455 5800 50  0001 C CNN
+	1    8455 5800
+	0    -1   -1   0
+$EndComp
+Text Label 6740 5335 1    50   ~ 0
+Vsensor
+Text Label 8205 5750 2    50   ~ 0
+SCL
+Text Label 8205 5650 2    50   ~ 0
+SDA
+Text Label 8205 5850 2    50   ~ 0
+GND
+Text Label 6940 5335 1    50   ~ 0
+GND
+Text Label 8205 5950 2    50   ~ 0
+Vsensor
+$Comp
+L neosensor_addon:ATECC508A J7
+U 1 1 60B67E25
 P 9685 5470
 F 0 "J7" H 9685 5837 50  0000 C CNN
-F 1 "78_01_030_0004" H 9685 5746 50  0000 C CNN
+F 1 "ATECC508A" H 9685 5746 50  0000 C CNN
 F 2 "neosensor_addon:ATECC508A" H 9685 5470 50  0001 L BNN
 F 3 "" H 9685 5470 50  0001 L BNN
@@
 	1    0    0    -1
 $EndComp
+Wire Wire Line
+	8600 2100 8600 2400
+Text Label 6840 5335 1    50   ~ 0
+GPIO0
+Text Label 8600 2400 3    50   ~ 0
+VDD
+$Comp
+L Regulator_Linear:AMS1117 U?
+U 1 1 60C3FD4D
+P 5035 5490
+F 0 "U?" H 5035 5732 50  0000 C CNN
+F 1 "AMS1117" H 5035 5641 50  0000 C CNN
+F 2 "Package_TO_SOT_SMD:SOT-223-3_TabPin2" H 5035 5690 50  0001 C CNN
+F 3 "http://www.advanced-monolithic.com/pdf/ds1117.pdf" H 5135 5240 50  0001 C CNN
+	1    5035 5490
+	1    0    0    -1
+$EndComp
+$Comp
+L Device:C C?
+U 1 1 60C4535A
+P 4480 5640
+F 0 "C?" H 4595 5686 50  0000 L CNN
+F 1 "100nF" H 4595 5595 50  0000 L CNN
+F 2 "" H 4518 5490 50  0001 C CNN
+F 3 "~" H 4480 5640 50  0001 C CNN
+	1    4480 5640
+	1    0    0    -1
+$EndComp
+Wire Wire Line
+	5335 5490 5410 5490
+$Comp
+L Device:C C?
+U 1 1 60C4A52B
+P 5410 5640
+F 0 "C?" H 5525 5686 50  0000 L CNN
+F 1 "C" H 5525 5595 50  0000 L CNN
+F 2 "" H 5448 5490 50  0001 C CNN
+F 3 "~" H 5410 5640 50  0001 C CNN
+	1    5410 5640
+	1    0    0    -1
+$EndComp
+Connection ~ 5410 5490
+Wire Wire Line
+	5410 5490 5520 5490
+Wire Wire Line
+	4480 5490 4735 5490
+Wire Wire Line
+	4480 5490 4240 5490
+Connection ~ 4480 5490
+Wire Wire Line
+	4480 5790 5035 5790
+Connection ~ 5035 5790
+Wire Wire Line
+	5035 5790 5410 5790
+Wire Wire Line
+	5035 5790 5035 5855
+Text Label 5035 5855 3    50   ~ 0
+GND
 $EndSCHEMATC

Commit message: mise a jour des schema
Parts:
- removed J7: ATECC508A, neosensor_addon:ATECC508A, symbol neosensor_addon:ATECC508A
- removed SW1: G71Y, neosensor_addon:G71Y_µsw_smd, symbol neOSensor-Cubecell_V1-rescue:G71Y-neosensor_addon-neOSensor_Cubecell_V1-rescue
- removed U1: HTCC-AB01, HTCC-AB01:htcc-ab01, symbol neOSensor-Cubecell_V1-rescue:HTCC-AB01-htcc-ab01-neOSensor_Cubecell_V1-rescue
- added C?: 1µF, symbol Device:C
- added IR?: IRsensor, neosensor_addon:IRsensor_TH_and_smd, symbol neosensor_addon:IRsensor
- added R? (x2): 15K, symbol Device:R
- added R?: R, symbol Device:R
- added SW1: G71Y, neosensor_addon:G71Y_µsw_smd, symbol neosensor_addon:G71Y
- added U1: HTCC-AB01, neosensor_addon:HTCC-AB01, symbol neosensor_addon:HTCC-AB01
- added U5: ATECC508A, neosensor_addon:SOIC-8_3.9x5.4mm_P1.27mm_HandSolder, symbol neosensor_addon:ATECC508A
- C2, C4: renamed from C?; footprint (none) -> Capacitor_SMD:C_0805_2012Metric_Pad1.15x1.40mm_HandSolder
- gave numbers to parts that had none: 1
Connections:
- net ADC: now also U1.12 (ADC)
- net GND: now also C?.2, R?.2, SW1.3, U1.1 (GND), U1.22 (GND), U1.5 (GND), U5.4 (GND)
- net GPIO0: now also U1.8 (GPIO0)
- net GPIO1: now also U1.13 (GPIO1)
- net GPIO2: now also U1.14 (GPIO2)
- net GPIO3: now also U1.15 (GPIO3)
- net GPIO4: now also U1.9 (GPIO4)
- net GPIO5: now also C?.1, R?.1, U1.10 (GPIO5)
- net MISO: now also U1.19 (MISO)
- net MOSI: now also U1.20 (MOSI)
- net RST: now also U1.11 (RST)
- net RX: now also U1.16 (RX)
- net SCK: now also U1.18 (SCK)
- net SCL: now also U1.6 (SCL), U5.6 (SCL)
- net SDA: now also U1.7 (SDA), U5.5 (SDA)
- net TX: now also U1.17 (TX)
- net VDD: now also JP1.3 (B), U1.3 (VDD); no longer JP1.1 (A)
- net VEXT: now also U1.4 (VEXT); no longer JP1.3 (B)
- net VIN: now also C2.1, U2.1 (V+), U4.3 (VI), U1.21 (VIN); no longer R1.2
- net VS*: now also U1.2 (VS*)
- net Vsensor: now also R1.2, IR?.1 (V+), U5.8 (VCC); no longer U2.1 (V+)
- net 3v3: now reaches C4.1, U4.2 (VO)
- net 3v3: now also JP1.1 (A), SW1.2
- new net: R?.1, R?.2, SW1.1
- no-connect marks 4 -> 0
Other:
- note removed: "ATECC508A-SSHDA"
- moved on the sheet: C2, C4, JP1, U2, U4

Commit message: update
Parts:
- removed C1, C3, C5, C6: 100n, Capacitor_SMD:C_0805_2012Metric_Pad1.15x1.40mm_HandSolder, symbol Device:C_Small
- removed C4: C, Capacitor_SMD:C_0805_2012Metric_Pad1.15x1.40mm_HandSolder, symbol Device:C
- removed R?: R, symbol Device:R
- added C3: 100µF, Capacitor_THT:CP_Radial_D5.0mm_P2.50mm, symbol Device:CP1_Small
- C1: renamed from C?; footprint (none) -> Resistor_SMD:R_0805_2012Metric_Pad1.20x1.40mm_HandSolder
- R4, R5: renamed from R?; footprint (none) -> Resistor_SMD:R_0805_2012Metric_Pad1.15x1.40mm_HandSolder
- gave numbers to parts that had none: 1
Connections:
- net GPIO0 is gone; now on net IR: U1.8 (GPIO0), U2.2 (OUT)
- net 3v3: now also C3.1; no longer SW1.2
- net GND: now also IR1.3 (GND), C3.2
- net VDD: no longer J2.1 (Pin_1)
- net VIN: no longer R2.2, U2.1 (V+)
- net Vsensor: now also J2.1 (Pin_1), R2.2, SW1.2, U2.1 (V+)
- net IR: now reaches IR1.2 (out)
Other:
- note added: "Expansion connectors for i2C sensors without interup"
- note removed: "Expansion connectors for i2C \nsensors without interup\n\n"
- moved on the sheet: C1, C2, IR1, J1, J2, J3, J5, J6, JP1, MH1, MH2, R4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

Commit message: update
Connections:
- net VIN: now also U2.1 (V+)
- net Vsensor: no longer U2.1 (V+)
Changed lines of the file:
@@
 $EndComp
 Text Label 6600 5200 1    50   ~ 0
-Vsensor
+VIN
 $Comp
 L Device:R R5
