File: pcb/lorawan-v2/_autosave-neosensoV5.sch (KiCad schematic (older format))
At the start: 43 parts, among them J1 Conn_01x04, J1 Conn_01x05, J2 Conn_01x04, J2 Conn_01x05, J3 Conn_01x04, J3 Conn_01x05, J4 Conn_01x05, J5 Conn_01x05, J6 Conn_01x04, Q1 2N7002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

Commit message: update
Parts:
- removed IR1: IRsensor, neosensor_addon:IRsensor_TH_and_smd, symbol neosensor_addon:IRsensor
- removed J1, J2, J5: Conn_01x05, Connector_PinHeader_2.54mm:PinHeader_1x05_P2.54mm_Vertical, symbol Connector_Generic:Conn_01x05
- removed J3, J6: Conn_01x04, Connector_PinHeader_2.54mm:PinHeader_1x04_P2.54mm_Vertical, symbol Connector_Generic:Conn_01x04
- removed JP1: SolderJumper_3_Bridged12, Jumper:SolderJumper-3_P1.3mm_Bridged2Bar12_Pad1.0x1.5mm, symbol Jumper:SolderJumper_3_Bridged12
- removed R1, R2: 10K, Resistor_SMD:R_0805_2012Metric_Pad1.15x1.40mm_HandSolder, symbol Device:R
- removed U1: HTCC-AB01, neosensor_addon:HTCC-AB01, symbol neosensor_addon:HTCC-AB01
- removed U5: ATECC508A, neosensor_addon:SOIC-8_3.9x5.4mm_P1.27mm_HandSolder, symbol neosensor_addon:ATECC508A
- added C3: 100nF, Resistor_SMD:R_0805_2012Metric_Pad1.20x1.40mm_HandSolder, symbol Device:C_Small
- added J6: Conn_01x06, Connector_PinHeader_2.54mm:PinHeader_1x06_P2.54mm_Vertical, symbol Connector_Generic:Conn_01x06
- added R13, R14, R15, R18: 22k, Resistor_SMD:R_0805_2012Metric_Pad1.20x1.40mm_HandSolder, symbol Device:R_Small
- added R16, R17, R19, R20: 33k, Resistor_SMD:R_0805_2012Metric_Pad1.20x1.40mm_HandSolder, symbol Device:R_Small
- added TP3: tp_an1, TestPoint:TestPoint_Loop_D2.50mm_Drill1.0mm, symbol Connector:TestPoint
- added TP4: tp_an0, TestPoint:TestPoint_Loop_D2.50mm_Drill1.0mm, symbol Connector:TestPoint
- added TP5: tp_an2, TestPoint:TestPoint_Loop_D2.50mm_Drill1.0mm, symbol Connector:TestPoint
- added TP6: tp_an3, TestPoint:TestPoint_Loop_D2.50mm_Drill1.0mm, symbol Connector:TestPoint
- added U5: LM2902, Package_SO:SO-14_5.3x10.2mm_P1.27mm, symbol Amplifier_Operational:LM2902
- SW3: renamed from SW1; value G71Y -> -
- renumbered IR2 to U1
Connections:
- net labels added: ANA_0, ANA_1, ANA_2, ANA_3
- net labels removed: GPIO1, GPIO2, GPIO3, GPIO4, GPIO5, MISO, MOSI, RST, RX, SCK, SW1, TX, VDD, VEXT, VIN, VS*, Vsensor
- wire segments 189 -> 191
Other:
- note added: "ANALOG inputs"
- note added: "HC-SR01 V+ accepts from 5 to 20v\nOUT pin is 3.3 TTL\n>> Remove R9 if IR sensor present <<"
- note added: "PIR sensor"
- note added: "Translate 5v analog input to 3v\n(NOT 3.3v due to ESP32 non linearity)\nV+ = 5v x 33k / 55k = 3v\nop. amp as follower"
- note removed: "Expansion connectors for i2C sensors with interup\n\n"
- note removed: "Expansion connectors for i2C sensors without interup"
- note removed: "HC-SR01 V+ accepts from 5 to 20v\nOUT pin is 3.3 TTL"
- note removed: "I2C crypto flash"
- note removed: "IR1 output is 100µA max\n+ R pull down needed (47K)"
- note removed: "PIR sensors"
- note removed: "Sensors power supply selector"
- note removed: "User push button"
- note removed: "either IR1 or IR2 (both is impossible)"
- moved on the sheet: C1, C2, C5, H1, H2, R11, R12, SW3, U1, U2, U4
