File: pcb/lorawan-v2/neOsensor-LoRaWANV2.sch (KiCad schematic (older format))
At the start: 43 parts, among them J1 Conn_01x04, J1 Conn_01x05, J2 Conn_01x04, J2 Conn_01x05, J3 Conn_01x04, J3 Conn_01x05, J4 Conn_01x05, J5 Conn_01x05, J6 Conn_01x04, Q1 2N7002, SW1 G71Y, SW1 clear, SW2 +, U1 HTCC-AB01, U2 OLED1.3_I2C, U3 ESP32_dev_30p, U4 AMS1117-3.3, U5 ATECC508A

Commit message: lorawanV2 schematic is ok. PCB is on way
Parts:
- removed C4: 1uF, Resistor_SMD:R_0805_2012Metric_Pad1.20x1.40mm_HandSolder, symbol Device:C_Small
- removed D1: Red, LED_SMD:LED_0805_2012Metric_Pad1.15x1.40mm_HandSolder, symbol Device:LED_Small_ALT
- removed J1, J2, J5: Conn_01x05, Connector_PinHeader_2.54mm:PinHeader_1x05_P2.54mm_Vertical, symbol Connector_Generic:Conn_01x05
- removed J3, J6: Conn_01x04, Connector_PinHeader_2.54mm:PinHeader_1x04_P2.54mm_Vertical, symbol Connector_Generic:Conn_01x04
- removed JP1: SolderJumper_3_Bridged12, Jumper:SolderJumper-3_P1.3mm_Bridged2Bar12_Pad1.0x1.5mm, symbol Jumper:SolderJumper_3_Bridged12
- removed Q1: 2N7002, Package_TO_SOT_SMD:SOT-23_Handsoldering, symbol Transistor_FET:2N7002
- removed R1, R2: 10K, Resistor_SMD:R_0805_2012Metric_Pad1.15x1.40mm_HandSolder, symbol Device:R
- removed R1: 150, Resistor_SMD:R_0805_2012Metric_Pad1.20x1.40mm_HandSolder, symbol Device:R_Small
- removed R10, R2, R7, R9: 15k, Resistor_SMD:R_0805_2012Metric_Pad1.20x1.40mm_HandSolder, symbol Device:R_Small
- removed R3: 470, Resistor_SMD:R_0805_2012Metric_Pad1.20x1.40mm_HandSolder, symbol Device:R_Small
- removed SW1: clear, neosensor_addon:G71Y_µsw_smd, symbol neosensor_addon:G71Y
- removed SW2: +, neosensor_addon:G71Y_µsw_smd, symbol neosensor_addon:G71Y
- removed U1: HTCC-AB01, neosensor_addon:HTCC-AB01, symbol neosensor_addon:HTCC-AB01
- removed U3: ESP32_dev_30p, neosensor_addon:ESP32_dev_30p, symbol neosensor_addon:ESP32_dev_30p
- added J2: Conn_01x02, Connector_PinHeader_2.54mm:PinHeader_1x02_P2.54mm_Vertical, symbol Connector_Generic:Conn_01x02
- added J7: Conn_01x05, Connector_PinHeader_2.54mm:PinHeader_1x05_P2.54mm_Vertical, symbol Connector_Generic:Conn_01x05
- added JP1: SolderJumper_3_Open, Jumper:SolderJumper-3_P1.3mm_Open_RoundedPad1.0x1.5mm, symbol Jumper:SolderJumper_3_Open
- added U4: HTCC-AB01, neosensor_addon:HTCC-AB01, symbol neosensor_addon:HTCC-AB01
- C1: renamed from C5; footprint Resistor_SMD:R_0805_2012Metric_Pad1.20x1.40mm_HandSolder -> Capacitor_SMD:C_0805_2012Metric_Pad1.15x1.40mm_HandSolder
- C2: renamed from C1; footprint Resistor_SMD:R_0805_2012Metric_Pad1.20x1.40mm_HandSolder -> Capacitor_SMD:C_0805_2012Metric_Pad1.15x1.40mm_HandSolder
- R1: renamed from R12; footprint Resistor_SMD:R_0805_2012Metric_Pad1.20x1.40mm_HandSolder -> Resistor_SMD:R_0805_2012Metric_Pad1.15x1.40mm_HandSolder
- R2: renamed from R11; footprint Resistor_SMD:R_0805_2012Metric_Pad1.20x1.40mm_HandSolder -> Resistor_SMD:R_0805_2012Metric_Pad1.15x1.40mm_HandSolder
- R3: renamed from R4; footprint Resistor_SMD:R_0805_2012Metric_Pad1.20x1.40mm_HandSolder -> Resistor_SMD:R_0805_2012Metric_Pad1.15x1.40mm_HandSolder
- R4: renamed from R8; footprint Resistor_SMD:R_0805_2012Metric_Pad1.20x1.40mm_HandSolder -> Resistor_SMD:R_0805_2012Metric_Pad1.15x1.40mm_HandSolder
- R5: footprint Resistor_SMD:R_0805_2012Metric_Pad1.20x1.40mm_HandSolder -> Resistor_SMD:R_0805_2012Metric_Pad1.15x1.40mm_HandSolder
- R6: renamed from R21; footprint Resistor_SMD:R_0805_2012Metric_Pad1.20x1.40mm_HandSolder -> Resistor_SMD:R_0805_2012Metric_Pad1.15x1.40mm_HandSolder
- renumbered C2 to C3, J2 to J3, J3 to J4, J4 to J5, J5 to J6, U2 to U1, U5 to U2, U4 to U3
Connections:
- net +5V is gone; now on net VIN: J6.1 (Pin_1)
- net RX2 is gone; now on net RX: J6.5 (Pin_5)
- net TX2 is gone; now on net TX: J6.4 (Pin_4), R5.1
- net +3V3: now also JP1.1 (A); no longer J1.1 (Pin_1), J3.1 (Pin_1), J4.1 (Pin_1), J5.1 (Pin_1), R3.2, R4.2, R6.2, U1.1 (VCC)
- net GND: now also J2.2 (Pin_2), J7.2 (Pin_2), U4.1 (GND), U4.22 (GND), U4.5 (GND)
- net INT: now also J7.5 (Pin_5), U4.13 (GPIO1)
- net PM_EN: now also U4.14 (GPIO2)
- net RX: now also U4.16 (RX)
- net SCL: now also J7.3 (Pin_3), U4.6 (SCL)
- net SDA: now also J7.4 (Pin_4), U4.7 (SDA)
- net SW1: now also U4.10 (GPIO5)
- net VDD: now also JP1.3 (B), U4.3 (VDD)
- net VIN: now also U4.21 (VIN)
- net Vsensor: now also J1.1 (Pin_1), J3.1 (Pin_1), J4.1 (Pin_1), J5.1 (Pin_1), R3.2, R4.2, R6.2, U1.1 (VCC), J7.1 (Pin_1), JP1.2 (C)
- net at R5.2: now also U4.17 (TX)
- new net VS+: J2.1 (Pin_1), U4.2 (VS*)
- no-connect marks 13 -> 9
Other:
- note added: "Notes:\n- ADC must be left floating to enable VBat reading\n (onboard BR1 not removed)\n"
- note added: "Solar panel"
- note added: "USB power"
- note added: "USB powered: junction 1-2\nSolar powered: junction 2-3 (AMS1117 not needed)"
- note added: "either IR1 or IR2 (both is not allowed)"
- note removed: "Expansion connectors for i2C sensors with interup\n\n"
- note removed: "Expansion connectors for i2C sensors without interup"
- note removed: "LED and SWITCHES"
- note removed: "Notes:\n- GPIO5 has a 10k pull-up on +3v3 on devkit V1 !!\n- GPIO5 reserved for Particule Meter ENable (3v3)\n- GPIOX reserved for LED + clear sw\n- GPIO13 reserved for noise sensor\n- GPIO4 reserved for IR sensor (input)\n- ADC2 pins cannot be used when WiFi in use\n- prefer ADC1 pins (GPIO32 --> 39)\n- GPIO1 & GPIO3 are serial0 (prog.)\n- GPIO2 onboard blue led @ devkit V1\n- EN must be floatin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"
- note removed: "Red led Vf=1.56v"
- note removed: "TODO:\n- remove R9\n- add 470R in serie withGPIO4 (IR input)"
- note removed: "either IR1 or IR2 (both is impossible)"
- moved on the sheet: C1, C2, C3, H1, H2, IR1, IR2, J1, J3, J4, J5, J6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

Commit message: lorawan-v2 pcb update
Parts:
- added R7: 47K, Resistor_SMD:R_0805_2012Metric_Pad1.15x1.40mm_HandSolder, symbol Device:R_Small
- added R8: 470, Resistor_SMD:R_0805_2012Metric_Pad1.15x1.40mm_HandSolder, symbol Device:R_Small
Connections:
- net GND: now also R7.1
- net IR: now also R7.2, R8.2
- net at U4.9 (GPIO4): now also R8.1
- no-connect marks 9 -> 8
Other:
- note added: "Notes:\n- ADC must be left floating to enable VBat reading\n (onboard BR1 not removed)\n- Panasonic IR sensor delivers upto 100µA, hence 47K"
- note removed: "Notes:\n- ADC must be left floating to enable VBat reading\n (onboard BR1 not removed)\n"
- moved on the sheet: R6
Changed lines of the file:
@@
 Power supply
 Text Notes 4250 2600 0    50   ~ 0
-Notes:\n- ADC must be left floating to enable VBat reading\n  (onboard BR1 not removed)\n
+Notes:\n- ADC must be left floating to enable VBat reading\n  (onboard BR1 not removed)\n- Panasonic IR sensor delivers upto 100µA, hence 47K
 $Comp
 L Device:C_Small C2
@@
 L Device:R_Small R6
 U 1 1 603D554C
-P 9475 3075
-F 0 "R6" V 9475 3075 50  0000 C CNN
-F 1 "15k" V 9500 2925 50  0000 C CNN
-F 2 "Resistor_SMD:R_0805_2012Metric_Pad1.15x1.40mm_HandSolder" H 9475 3075 50  0001 C CNN
-F 3 "~" H 9475 3075 50  0001 C CNN
-	1    9475 3075
+P 9375 3075
+F 0 "R6" V 9375 3075 50  0000 C CNN
+F 1 "15k" V 9400 2925 50  0000 C CNN
+F 2 "Resistor_SMD:R_0805_2012Metric_Pad1.15x1.40mm_HandSolder" H 9375 3075 50  0001 C CNN
+F 3 "~" H 9375 3075 50  0001 C CNN
+	1    9375 3075
 	-1   0    0    1
 $EndComp
-Text Label 7400 2900 0    50   ~ 0
+Text Label 6600 2900 0    50   ~ 0
 SCL
-Text Label 7400 3000 0    50   ~ 0
+Text Label 6700 3000 0    50   ~ 0
 SDA
 Wire Wire Line
@@
 Vsensor
 Wire Wire Line
-	9475 2975 9475 2750
-Wire Wire Line
-	9475 2750 9775 2750
-Text Label 9775 2750 2    50   ~ 0
+	9375 2975 9375 2750
+Wire Wire Line
+	9375 2750 9675 2750
+Text Label 9675 2750 2    50   ~ 0
 Vsensor
 Wire Wire Line
-	9475 3300 9475 3175
-Wire Wire Line
-	8700 3300 9475 3300
-Text Label 9000 3300 2    50   ~ 0
+	9375 3300 9375 3175
+Text Label 9675 3300 2    50   ~ 0
 INT
 NoConn ~ 7700 3100
-NoConn ~ 7700 3200
 Wire Wire Line
 	7400 3300 7700 3300
@@
 Text Label 5950 1425 0    50   ~ 0
 INT
+Wire Wire Line
+	8700 3300 9375 3300
+Wire Wire Line
+	9675 3300 9375 3300
+Connection ~ 9375 3300
+Wire Wire Line
+	6700 3000 7000 3000
+Connection ~ 7000 3000
+Wire Wire Line
+	6600 2900 6900 2900
+Connection ~ 6900 2900
+$Comp
+L Device:R_Small R8
+U 1 1 60C35398
+P 7500 3200
+F 0 "R8" V 7500 3200 50  0000 C CNN
+F 1 "470" V 7425 3200 50  0000 C CNN
+F 2 "Resistor_SMD:R_0805_2012Metric_Pad1.15x1.40mm_HandSolder" H 7500 3200 50  0001 C CNN
+F 3 "~" H 7500 3200 50  0001 C CNN
+	1    7500 3200
+	0    1    1    0
+$EndComp
+Wire Wire Line
+	7700 3200 7600 3200
+Text Label 7000 3200 0    50   ~ 0
+IR
+$Comp
+L Device:R_Small R7
+U 1 1 60C3D53E
+P 7275 3475
+F 0 "R7" V 7275 3475 50  0000 C CNN
+F 1 "47K" V 7200 3475 50  0000 C CNN
+F 2 "Resistor_SMD:R_0805_2012Metric_Pad1.15x1.40mm_HandSolder" H 7275 3475 50  0001 C CNN
+F 3 "~" H 7275 3475 50  0001 C CNN
+	1    7275 3475
+	-1   0    0    1
+$EndComp
+Wire Wire Line
+	7275 3375 7275 3200
+$Comp
+L power:GND #PWR0101
+U 1 1 60C41A48
+P 7275 3650
+F 0 "#PWR0101" H 7275 3400 50  0001 C CNN
+F 1 "GND" H 7280 3477 50  0000 C CNN
+F 2 "" H 7275 3650 50  0001 C CNN
+F 3 "" H 7275 3650 50  0001 C CNN
+	1    7275 3650
+	1    0    0    -1
+$EndComp
+Wire Wire Line
+	7275 3650 7275 3575
+Connection ~ 7275 3200
+Wire Wire Line
+	7275 3200 7400 3200
+Wire Wire Line
+	7000 3200 7275 3200
 $EndSCHEMATC

Commit message: update
Parts:
- removed J4: Conn_01x05, Connector_PinHeader_2.54mm:PinHeader_1x05_P2.54mm_Vertical, symbol Connector_Generic:Conn_01x05
- added C4: 100n, Capacitor_SMD:C_0805_2012Metric_Pad1.18x1.45mm_HandSolder, symbol Device:C_Small
- added J4: Conn_01x04, Connector_PinHeader_2.54mm:PinHeader_1x04_P2.54mm_Vertical, symbol Connector_Generic:Conn_01x04
Connections:
- net GND: now also C4.1, J4.2 (Pin_2)
- net SCL: now also J4.3 (Pin_3)
- net SDA: now also J4.4 (Pin_4)
- net Vsensor: now also C4.2, J4.1 (Pin_1)
Other:
- moved on the sheet: J7
Changed lines of the file:
@@
 I2C crypto flash
 Wire Wire Line
-	850  1600 1100 1600
+	850  1600 1075 1600
 Text Label 850  1600 0    50   ~ 0
 GND
@@
 SCL
 Wire Wire Line
-	1925 1300 1700 1300
+	1925 1300 1750 1300
 Text Label 1925 1300 0    50   ~ 0
 Vsensor
-Wire Notes Line
-	2400 625  2400 1875
-Wire Notes Line
-	2400 1875 600  1875
 Wire Notes Line
 	6850 6550 4700 6550
@@
 $EndComp
 $Comp
-L Connector_Generic:Conn_01x05 J4
-U 1 1 601CACB8
-P 7350 1225
-F 0 "J4" H 7300 1525 50  0000 L CNN
-F 1 "Conn_01x05" H 7150 925 50  0000 L CNN
-F 2 "Connector_PinHeader_2.54mm:PinHeader_1x05_P2.54mm_Vertical" H 7350 1225 50  0001 C CNN
-F 3 "~" H 7350 1225 50  0001 C CNN
-	1    7350 1225
-	1    0    0    -1
-$EndComp
-$Comp
 L Connector_Generic:Conn_01x05 J5
 U 1 1 601CBCDB
@@
 SDA
 Wire Wire Line
-	7150 1025 6850 1025
-Text Label 6850 1025 0    50   ~ 0
-Vsensor
-Wire Wire Line
-	6850 1125 7150 1125
-Text Label 6850 1125 0    50   ~ 0
-GND
-Wire Wire Line
-	6850 1225 7150 1225
-Text Label 6850 1225 0    50   ~ 0
+	6175 1025 5875 1025
+Text Label 5875 1025 0    50   ~ 0
+Vsensor
+Wire Wire Line
+	5875 1125 6175 1125
+Text Label 5875 1125 0    50   ~ 0
+GND
+Wire Wire Line
+	5875 1225 6175 1225
+Text Label 5875 1225 0    50   ~ 0
 SCL
 Wire Wire Line
-	6850 1325 7150 1325
-Text Label 6850 1325 0    50   ~ 0
+	5875 1325 6175 1325
+Text Label 5875 1325 0    50   ~ 0
 SDA
 Wire Wire Line
@@
 SDA
 Wire Wire Line
-	6850 1425 7150 1425
-Wire Wire Line
 	7800 1425 8100 1425
 Text Label 7800 1425 0    50   ~ 0
-INT
-Text Label 6850 1425 0    50   ~ 0
 INT
 Wire Wire Line
@@
 L Connector_Generic:Conn_01x05 J7
 U 1 1 60D63244
-P 6450 1225
-F 0 "J7" H 6400 1525 50  0000 L CNN
-F 1 "Conn_01x05" H 6250 925 50  0000 L CNN
-F 2 "Connector_PinHeader_2.54mm:PinHeader_1x05_P2.54mm_Vertical" H 6450 1225 50  0001 C CNN
-F 3 "~" H 6450 1225 50  0001 C CNN
-	1    6450 1225
-	1    0    0    -1
-$EndComp
-Wire Wire Line
-	6250 1025 5950 1025
-Text Label 5950 1025 0    50   ~ 0
-Vsensor
-Wire Wire Line
-	5950 1125 6250 1125
-Text Label 5950 1125 0    50   ~ 0
-GND
-Wire Wire Line
-	5950 1225 6250 1225
-Text Label 5950 1225 0    50   ~ 0
+P 7500 1225
+F 0 "J7" H 7450 1525 50  0000 L CNN
+F 1 "Conn_01x05" H 7300 925 50  0000 L CNN
+F 2 "Connector_PinHeader_2.54mm:PinHeader_1x05_P2.54mm_Vertical" H 7500 1225 50  0001 C CNN
+F 3 "~" H 7500 1225 50  0001 C CNN
+	1    7500 1225
+	1    0    0    -1
+$EndComp
+Wire Wire Line
+	7300 1025 7000 1025
+Text Label 7000 1025 0    50   ~ 0
+Vsensor
+Wire Wire Line
+	7000 1125 7300 1125
+Text Label 7000 1125 0    50   ~ 0
+GND
+Wire Wire Line
+	7000 1225 7300 1225
+Text Label 7000 1225 0    50   ~ 0
 SCL
 Wire Wire Line
-	5950 1325 6250 1325
-Text Label 5950 1325 0    50   ~ 0
+	7000 1325 7300 1325
+Text Label 7000 1325 0    50   ~ 0
 SDA
 Wire Wire Line
-	5950 1425 6250 1425
-Text Label 5950 1425 0    50   ~ 0
+	7000 1425 7300 1425
+Text Label 7000 1425 0    50   ~ 0
 INT
 Wire Wire Line
@@
 Wire Wire Line
 	7000 3200 7275 3200
+$Comp
+L Connector_Generic:Conn_01x04 J4
+U 1 1 60C16F38
+P 6375 1125
+F 0 "J4" H 6325 1325 50  0000 L CNN
+F 1 "Conn_01x04" H 6175 825 50  0000 L CNN
+F 2 "Connector_PinHeader_2.54mm:PinHeader_1x04_P2.54mm_Vertical" H 6375 1125 50  0001 C CNN
+F 3 "~" H 6375 1125 50  0001 C CNN
+	1    6375 1125
+	1    0    0    -1
+$EndComp
+$Comp
+L Device:C_Small C4
+U 1 1 60C48C70
+P 1425 1850
+F 0 "C4" V 1325 1975 50  0000 C CNN
+F 1 "100n" V 1325 1700 50  0000 C CNN
+F 2 "Capacitor_SMD:C_0805_2012Metric_Pad1.18x1.45mm_HandSolder" H 1425 1850 50  0001 C CNN
+F 3 "~" H 1425 1850 50  0001 C CNN
+	1    1425 1850
+	0    -1   -1   0
+$EndComp
+Wire Wire Line
+	1325 1850 1075 1850
+Wire Wire Line
+	1075 1850 1075 1600
+Connection ~ 1075 1600
+Wire Wire Line
+	1075 1600 1100 1600
+Wire Wire Line
+	1525 1850 1750 1850
+Wire Wire Line
+	1750 1850 1750 1300
+Connection ~ 1750 1300
+Wire Wire Line
+	1750 1300 1700 1300
 $EndSCHEMATC

Commit message: lorawanV2 docs update
Other:
- note added: "- set battery connector JST xxx\n- M3 holes not aligned !!\n"
- note added: ">>> TODO: LoRaWAN V2.1 <<<"
Changed lines of the file:
@@
 Wire Wire Line
 	1750 1300 1700 1300
+Wire Notes Line
+	3200 2875 6125 2875
+Wire Notes Line
+	6125 2875 6125 4275
+Wire Notes Line
+	6125 4275 3200 4275
+Wire Notes Line
+	3200 4275 3200 2875
+Text Notes 3250 3025 0    71   ~ 14
+>>> TODO: LoRaWAN V2.1 <<<
+Text Notes 3250 3200 0    50   ~ 0
+- set battery connector JST xxx\n- M3 holes not aligned !!\n
 $EndSCHEMATC

Commit message: update
Parts:
- C2: value 100nF -> 100n
Changed lines of the file:
@@
 P 6975 5700
 F 0 "C2" H 7067 5746 50  0000 L CNN
-F 1 "100nF" H 7067 5655 50  0000 L CNN
+F 1 "100n" H 7067 5655 50  0000 L CNN
 F 2 "Capacitor_SMD:C_0805_2012Metric_Pad1.15x1.40mm_HandSolder" H 6975 5700 50  0001 C CNN
 F 3 "~" H 6975 5700 50  0001 C CNN

Commit message: update
Other:
- note added: "- set battery connector JST xxx\n- M3 holes not aligned !!\n- [done] R4 silk to move"
- note removed: "- set battery connector JST xxx\n- M3 holes not aligned !!\n"
Changed lines of the file:
@@
 >>> TODO: LoRaWAN V2.1 <<<
 Text Notes 3250 3200 0    50   ~ 0
-- set battery connector JST xxx\n- M3 holes not aligned !!\n
+- set battery connector JST xxx\n- M3 holes not aligned !!\n- [done] R4 silk to move
 $EndSCHEMATC

Commit message: update
Other:
- note added: "- set battery connector JST xxx\n- M3 holes not aligned !!\n- [done] R4 silk to move\n- name Jx pins@PCB (e.g SDA, SCL ...)"
- note removed: "- set battery connector JST xxx\n- M3 holes not aligned !!\n- [done] R4 silk to move"
Changed lines of the file:
@@
 Text Notes 3250 3025 0    71   ~ 14
 >>> TODO: LoRaWAN V2.1 <<<
-Text Notes 3250 3200 0    50   ~ 0
-- set battery connector JST xxx\n- M3 holes not aligned !!\n- [done] R4 silk to move
+Text Notes 3275 3475 0    50   ~ 0
+- set battery connector JST xxx\n- M3 holes not aligned !!\n- [done] R4 silk to move\n- name Jx pins@PCB (e.g SDA, SCL ...)
 $EndSCHEMATC

Commit message: update
Other:
- note added: "- set battery connector JST xxx\n- VS+ / GND to invert (JSTxxx connector)\n- M3 holes not aligned !!\n- [done] R4 silk to move\n- name Jx pins@PCB (e.g SDA, SCL ...)"
- note removed: "- set battery connector JST xxx\n- M3 holes not aligned !!\n- [done] R4 silk to move\n- name Jx pins@PCB (e.g SDA, SCL ...)"
Changed lines of the file:
@@
 >>> TODO: LoRaWAN V2.1 <<<
 Text Notes 3275 3475 0    50   ~ 0
-- set battery connector JST xxx\n- M3 holes not aligned !!\n- [done] R4 silk to move\n- name Jx pins@PCB (e.g SDA, SCL ...)
+- set battery connector JST xxx\n- VS+ / GND to invert (JSTxxx connector)\n- M3 holes not aligned !!\n- [done] R4 silk to move\n- name Jx pins@PCB (e.g SDA, SCL ...)
 $EndSCHEMATC
