File: pcb/lorawan-v2/neOsensor-LoRaWANV2.sch (KiCad schematic (older format))
At the start: 29 parts, among them J1 Conn_01x04, J2 Conn_01x02, J3 Conn_01x04, J4 Conn_01x04, J5 Conn_01x05, J6 Conn_01x05, J7 Conn_01x05, SW1 G71Y, U1 OLED1.3_I2C, U2 ATECC508A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

Commit message: update
Parts:
- removed J3: Conn_01x04, Connector_PinHeader_2.54mm:PinHeader_1x04_P2.54mm_Vertical, symbol Connector_Generic:Conn_01x04
- added J3: Conn_01x05, Connector_PinHeader_2.54mm:PinHeader_1x05_P2.54mm_Vertical, symbol Connector_Generic:Conn_01x05
Connections:
- net GND: now also J3.2 (Pin_2)
- net INT: now also U4.8 (GPIO0), J3.5 (Pin_5); no longer U4.13 (GPIO1)
- net PM_EN: now also U4.10 (GPIO4); no longer U4.14 (GPIO2)
- net SCL: now also J3.3 (Pin_3)
- net SDA: now also J3.4 (Pin_4)
- net SW1: now also U4.13 (GPIO1); no longer U4.10 (GPIO4)
- net Vsensor: now also J3.1 (Pin_1)
- no-connect marks 8 -> 9
Other:
- note added: "- set battery connector JST xxx\n- VS+ / GND to invert (JSTxxx connector)\n- M3 holes not aligned !!\n- [done] R4 silk to move\n- GPIO4 is also used to drive the onboard led\n- @PCB C3: + sign bigger !!\n- J1 or J4: add INT pin\n- J3: add INT pin\n- @PCB J1 or J4: flip (to have both config). Check TSL2561 fits to front\n- name Jx pins@PCB (e.g SDA, SCL ...)\n- ERROR GPIO4 and 5 swapped --> model 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"
- note added: "Notes:\n- ADC must be left floating to enable VBat reading\n (onboard BR1 not removed)\n- to READ Vbat ==> activate GPIO7 but BEWARE NOT TO\n PRESS USER button at the same time !!!\n- Panasonic IR sensor delivers upto 100µA, hence 47K\n- GPIO0 at powerup: if GND --> bootloader mode"
- note removed: "- set battery connector JST xxx\n- VS+ / GND to invert (JSTxxx connector)\n- M3 holes not aligned !!\n- [done] R4 silk to move\n- @PCB C3: + sign bigger !!\n- J1 or J4: add INT pin\n- @PCB J1 or J4: flip (to have both config). Check TSL2561 fits to front\n- name Jx pins@PCB (e.g SDA, SCL ...)\n- add Conn_01x02 on GPIO0 (force bootloader enable)"
- note removed: "Notes:\n- ADC must be left floating to enable VBat reading\n (onboard BR1 not removed)\n- Panasonic IR sensor delivers upto 100µA, hence 47K"
- moved on the sheet: J4, R6
Changed lines of the file:
@@
 encoding utf-8
 Sheet 1 1
-Title "neOSensor-LoRaWAN V2"
-Date "2021-06-08"
-Rev "2"
+Title "neOSensor-LoRaWAN V2.1"
+Date "2021-07-01"
+Rev "2.1"
 Comp "(c) neOCampus / Dr THIEBOLT François"
 Comment1 "Univ.Tlse3 / IRIT / neOCampus"
@@
 Text Label 4150 1325 0    50   ~ 0
 SDA
-$Comp
-L Connector_Generic:Conn_01x04 J3
-U 1 1 601D570B
-P 5500 1125
-F 0 "J3" H 5450 1325 50  0000 L CNN
-F 1 "Conn_01x04" H 5300 825 50  0000 L CNN
-F 2 "Connector_PinHeader_2.54mm:PinHeader_1x04_P2.54mm_Vertical" H 5500 1125 50  0001 C CNN
-F 3 "~" H 5500 1125 50  0001 C CNN
-	1    5500 1125
-	1    0    0    -1
-$EndComp
-Wire Wire Line
-	5300 1025 5000 1025
-Text Label 5000 1025 0    50   ~ 0
-Vsensor
-Wire Wire Line
-	5000 1125 5300 1125
-Text Label 5000 1125 0    50   ~ 0
-GND
-Wire Wire Line
-	5000 1225 5300 1225
-Text Label 5000 1225 0    50   ~ 0
+Wire Wire Line
+	6350 1025 6050 1025
+Text Label 6050 1025 0    50   ~ 0
+Vsensor
+Wire Wire Line
+	6050 1125 6350 1125
+Text Label 6050 1125 0    50   ~ 0
+GND
+Wire Wire Line
+	6050 1225 6350 1225
+Text Label 6050 1225 0    50   ~ 0
 SCL
 Wire Wire Line
-	5000 1325 5300 1325
-Text Label 5000 1325 0    50   ~ 0
+	6050 1325 6350 1325
+Text Label 6050 1325 0    50   ~ 0
 SDA
 Wire Wire Line
-	6175 1025 5875 1025
-Text Label 5875 1025 0    50   ~ 0
-Vsensor
-Wire Wire Line
-	5875 1125 6175 1125
-Text Label 5875 1125 0    50   ~ 0
-GND
-Wire Wire Line
-	5875 1225 6175 1225
-Text Label 5875 1225 0    50   ~ 0
+	5375 1025 5075 1025
+Text Label 5075 1025 0    50   ~ 0
+Vsensor
+Wire Wire Line
+	5075 1125 5375 1125
+Text Label 5075 1125 0    50   ~ 0
+GND
+Wire Wire Line
+	5075 1225 5375 1225
+Text Label 5075 1225 0    50   ~ 0
 SCL
 Wire Wire Line
-	5875 1325 6175 1325
-Text Label 5875 1325 0    50   ~ 0
+	5075 1325 5375 1325
+Text Label 5075 1325 0    50   ~ 0
 SDA
 Wire Wire Line
@@
 P 6900 2650
 F 0 "R3" V 6900 2650 50  0000 C CNN
-F 1 "4K7" V 6925 2500 50  0000 C CNN
+F 1 "4K7" V 6950 2475 50  0000 C CNN
 F 2 "Resistor_SMD:R_0805_2012Metric_Pad1.15x1.40mm_HandSolder" H 6900 2650 50  0001 C CNN
 F 3 "~" H 6900 2650 50  0001 C CNN
@@
 P 7000 2650
 F 0 "R4" V 7000 2650 50  0000 C CNN
-F 1 "4K7" V 7025 2500 50  0000 C CNN
+F 1 "4K7" V 7050 2475 50  0000 C CNN
 F 2 "Resistor_SMD:R_0805_2012Metric_Pad1.15x1.40mm_HandSolder" H 7000 2650 50  0001 C CNN
 F 3 "~" H 7000 2650 50  0001 C CNN
@@
 Text Notes 6250 4800 0    100  ~ 0
 Power supply
-Text Notes 4250 2600 0    50   ~ 0
-Notes:\n- ADC must be left floating to enable VBat reading\n  (onboard BR1 not removed)\n- Panasonic IR sensor delivers upto 100µA, hence 47K
+Text Notes 3400 2150 0    50   ~ 0
+Notes:\n- ADC must be left floating to enable VBat reading\n  (onboard BR1 not removed)\n- to READ Vbat ==> activate GPIO7 but BEWARE NOT TO\n    PRESS USER button at the same time !!!\n- Panasonic IR sensor delivers upto 100µA, hence 47K\n- GPIO0 at powerup: if GND --> bootloader mode
 $Comp
 L Device:C_Small C2
@@
 U 1 1 60CE8BBB
 P 8200 2900
-F 0 "U4" H 8200 3665 50  0000 C CNN
-F 1 "HTCC-AB01" H 8200 3574 50  0000 C CNN
+F 0 "U4" H 7850 3775 50  0000 C CNN
+F 1 "HTCC-AB01" H 8200 2275 50  0000 C CNN
 F 2 "neosensor_addon:HTCC-AB01" V 8200 2900 50  0001 C CIN
 F 3 "" H 7900 2300 50  0001 C CNN
@@
 L Device:R_Small R6
 U 1 1 603D554C
-P 9375 3075
-F 0 "R6" V 9375 3075 50  0000 C CNN
-F 1 "15k" V 9400 2925 50  0000 C CNN
-F 2 "Resistor_SMD:R_0805_2012Metric_Pad1.15x1.40mm_HandSolder" H 9375 3075 50  0001 C CNN
-F 3 "~" H 9375 3075 50  0001 C CNN
-	1    9375 3075
+P 7125 2650
+F 0 "R6" V 7125 2650 50  0000 C CNN
+F 1 "15k" V 7175 2475 50  0000 C CNN
+F 2 "Resistor_SMD:R_0805_2012Metric_Pad1.15x1.40mm_HandSolder" H 7125 2650 50  0001 C CNN
+F 3 "~" H 7125 2650 50  0001 C CNN
+	1    7125 2650
 	-1   0    0    1
 $EndComp
@@
 Vsensor
 Wire Wire Line
-	9375 2975 9375 2750
-Wire Wire Line
-	9375 2750 9675 2750
-Text Label 9675 2750 2    50   ~ 0
-Vsensor
-Wire Wire Line
-	9375 3300 9375 3175
-Text Label 9675 3300 2    50   ~ 0
-INT
-NoConn ~ 7700 3100
-Wire Wire Line
 	7400 3300 7700 3300
-Text Label 7400 3300 0    50   ~ 0
-SW1
-Text Label 9000 3200 2    50   ~ 0
-PM_EN
 $Comp
 L power:PWR_FLAG #FLG0101
@@
 Text Label 3450 7325 1    50   ~ 0
 VIN
-Wire Wire Line
-	9000 3200 8700 3200
 $Comp
 L power:PWR_FLAG #FLG0105
@@
 INT
 Wire Wire Line
-	8700 3300 9375 3300
-Wire Wire Line
-	9675 3300 9375 3300
-Connection ~ 9375 3300
-Wire Wire Line
 	6700 3000 7000 3000
 Connection ~ 7000 3000
@@
 P 7500 3200
 F 0 "R8" V 7500 3200 50  0000 C CNN
-F 1 "470" V 7425 3200 50  0000 C CNN
+F 1 "470" V 7450 3050 50  0000 C CNN
 F 2 "Resistor_SMD:R_0805_2012Metric_Pad1.15x1.40mm_HandSolder" H 7500 3200 50  0001 C CNN
 F 3 "~" H 7500 3200 50  0001 C CNN
@@
 L Connector_Generic:Conn_01x04 J4
 U 1 1 60C16F38
-P 6375 1125
-F 0 "J4" H 6325 1325 50  0000 L CNN
-F 1 "Conn_01x04" H 6175 825 50  0000 L CNN
-F 2 "Connector_PinHeader_2.54mm:PinHeader_1x04_P2.54mm_Vertical" H 6375 1125 50  0001 C CNN
-F 3 "~" H 6375 1125 50  0001 C CNN
-	1    6375 1125
+P 5575 1125
+F 0 "J4" H 5525 1325 50  0000 L CNN
+F 1 "Conn_01x04" H 5375 825 50  0000 L CNN
+F 2 "Connector_PinHeader_2.54mm:PinHeader_1x04_P2.54mm_Vertical" H 5575 1125 50  0001 C CNN
+F 3 "~" H 5575 1125 50  0001 C CNN
+	1    5575 1125
 	1    0    0    -1
 $EndComp
@@
 Text Notes 3250 3025 0    71   ~ 14
 >>> TODO: LoRaWAN V2.1 <<<
-Text Notes 3200 3750 0    50   ~ 0
-- set battery connector JST xxx\n- VS+ / GND to invert (JSTxxx connector)\n- M3 holes not aligned !!\n- [done] R4 silk to move\n- @PCB C3: + sign bigger !!\n- J1 or J4: add INT pin\n- @PCB J1 or J4: flip (to have both config). Check TSL2561 fits to front\n- name Jx pins@PCB (e.g SDA, SCL ...)\n- add Conn_01x02 on GPIO0 (force bootloader enable)
+Text Notes 3200 4050 0    50   ~ 0
+- set battery connector JST xxx\n- VS+ / GND to invert (JSTxxx connector)\n- M3 holes not aligned !!\n- [done] R4 silk to move\n- GPIO4 is also used to drive the onboard led\n- @PCB C3: + sign bigger !!\n- J1 or J4: add INT pin\n- J3: add INT pin\n- @PCB J1 or J4: flip (to have both config). Check TSL2561 fits to front\n- name Jx pins@PCB (e.g SDA, SCL ...)\n- ERROR GPIO4 and 5 swapped --> model corrected, apply to PCB\n- add Conn_01x02 on GPIO0 (force bootloader enable)
+Wire Wire Line
+	7000 2350 7125 2350
+Wire Wire Line
+	7125 2350 7125 2550
+Connection ~ 7000 2350
+Wire Wire Line
+	6800 3100 7125 3100
+Wire Wire Line
+	7125 2750 7125 3100
+Connection ~ 7125 3100
+Wire Wire Line
+	7125 3100 7700 3100
+Text Label 6800 3100 0    50   ~ 0
+INT
+Text Label 7400 3300 0    50   ~ 0
+PM_EN
+Wire Wire Line
+	9000 3300 8700 3300
+Text Label 9000 3300 2    50   ~ 0
+SW1
+NoConn ~ 8700 3200
+NoConn ~ 3750 3600
+$Comp
+L Connector_Generic:Conn_01x05 J3
+U 1 1 60E126AF
+P 6550 1225
+F 0 "J3" H 6500 1525 50  0000 L CNN
+F 1 "Conn_01x05" H 6325 925 50  0000 L CNN
+F 2 "Connector_PinHeader_2.54mm:PinHeader_1x05_P2.54mm_Vertical" H 6550 1225 50  0001 C CNN
+F 3 "~" H 6550 1225 50  0001 C CNN
+	1    6550 1225
+	1    0    0    -1
+$EndComp
+Wire Wire Line
+	6050 1425 6350 1425
+Text Label 6050 1425 0    50   ~ 0
+INT
 $EndSCHEMATC

Commit message: update
Parts:
- removed J1: Conn_01x04, Connector_PinHeader_2.54mm:PinHeader_1x04_P2.54mm_Vertical, symbol Connector_Generic:Conn_01x04
- added J1: Conn_01x05, Connector_PinHeader_2.54mm:PinHeader_1x05_P2.54mm_Vertical, symbol Connector_Generic:Conn_01x05
- J2: footprint Connector_PinHeader_2.54mm:PinHeader_1x02_P2.54mm_Vertical -> Connector_JST:JST_PH_S2B-PH-K_1x02_P2.00mm_Horizontal
Connections:
- net GND: now also J1.2 (Pin_2)
- net INT: now also J1.5 (Pin_5)
- net SCL: now also J1.3 (Pin_3)
- net SDA: now also J1.4 (Pin_4)
- net Vsensor: now also J1.1 (Pin_1)
Other:
- note added: "JST PH 2.0mm connector"
- moved on the sheet: J2, J3, J4, J5, J6, J7
Changed lines of the file:
@@
 +3V3
-$Comp
-L Connector_Generic:Conn_01x04 J1
-U 1 1 601C66E2
-P 4650 1125
-F 0 "J1" H 4600 1325 50  0000 L CNN
-F 1 "Conn_01x04" H 4450 825 50  0000 L CNN
-F 2 "Connector_PinHeader_2.54mm:PinHeader_1x04_P2.54mm_Vertical" H 4650 1125 50  0001 C CNN
-F 3 "~" H 4650 1125 50  0001 C CNN
-	1    4650 1125
-	1    0    0    -1
-$EndComp
 $Comp
 L Connector_Generic:Conn_01x05 J5
 U 1 1 601CBCDB
-P 8300 1225
-F 0 "J5" H 8250 1525 50  0000 L CNN
-F 1 "Conn_01x05" H 8100 925 50  0000 L CNN
-F 2 "Connector_PinHeader_2.54mm:PinHeader_1x05_P2.54mm_Vertical" H 8300 1225 50  0001 C CNN
-F 3 "~" H 8300 1225 50  0001 C CNN
-	1    8300 1225
+P 8300 1200
+F 0 "J5" H 8250 1500 50  0000 L CNN
+F 1 "Conn_01x05" H 8100 900 50  0000 L CNN
+F 2 "Connector_PinHeader_2.54mm:PinHeader_1x05_P2.54mm_Vertical" H 8300 1200 50  0001 C CNN
+F 3 "~" H 8300 1200 50  0001 C CNN
+	1    8300 1200
 	1    0    0    -1
 $EndComp
@@
 	7425 5900 7425 5750
 Wire Wire Line
-	4450 1025 4150 1025
-Text Label 4150 1025 0    50   ~ 0
-Vsensor
-Wire Wire Line
-	4150 1125 4450 1125
-Text Label 4150 1125 0    50   ~ 0
-GND
-Wire Wire Line
-	4150 1225 4450 1225
-Text Label 4150 1225 0    50   ~ 0
+	4450 1000 4150 1000
+Text Label 4150 1000 0    50   ~ 0
+Vsensor
+Wire Wire Line
+	4150 1100 4450 1100
+Text Label 4150 1100 0    50   ~ 0
+GND
+Wire Wire Line
+	4150 1200 4450 1200
+Text Label 4150 1200 0    50   ~ 0
 SCL
 Wire Wire Line
-	4150 1325 4450 1325
-Text Label 4150 1325 0    50   ~ 0
+	4150 1300 4450 1300
+Text Label 4150 1300 0    50   ~ 0
 SDA
 Wire Wire Line
-	6350 1025 6050 1025
-Text Label 6050 1025 0    50   ~ 0
-Vsensor
-Wire Wire Line
-	6050 1125 6350 1125
-Text Label 6050 1125 0    50   ~ 0
-GND
-Wire Wire Line
-	6050 1225 6350 1225
-Text Label 6050 1225 0    50   ~ 0
+	6350 1000 6050 1000
+Text Label 6050 1000 0    50   ~ 0
+Vsensor
+Wire Wire Line
+	6050 1100 6350 1100
+Text Label 6050 1100 0    50   ~ 0
+GND
+Wire Wire Line
+	6050 1200 6350 1200
+Text Label 6050 1200 0    50   ~ 0
 SCL
 Wire Wire Line
-	6050 1325 6350 1325
-Text Label 6050 1325 0    50   ~ 0
+	6050 1300 6350 1300
+Text Label 6050 1300 0    50   ~ 0
 SDA
 Wire Wire Line
-	5375 1025 5075 1025
-Text Label 5075 1025 0    50   ~ 0
-Vsensor
-Wire Wire Line
-	5075 1125 5375 1125
-Text Label 5075 1125 0    50   ~ 0
-GND
-Wire Wire Line
-	5075 1225 5375 1225
-Text Label 5075 1225 0    50   ~ 0
+	5375 1000 5075 1000
+Text Label 5075 1000 0    50   ~ 0
+Vsensor
+Wire Wire Line
+	5075 1100 5375 1100
+Text Label 5075 1100 0    50   ~ 0
+GND
+Wire Wire Line
+	5075 1200 5375 1200
+Text Label 5075 1200 0    50   ~ 0
 SCL
 Wire Wire Line
-	5075 1325 5375 1325
-Text Label 5075 1325 0    50   ~ 0
+	5075 1300 5375 1300
+Text Label 5075 1300 0    50   ~ 0
 SDA
 Wire Wire Line
-	8100 1025 7800 1025
-Text Label 7800 1025 0    50   ~ 0
-Vsensor
-Wire Wire Line
-	7800 1125 8100 1125
-Text Label 7800 1125 0    50   ~ 0
-GND
-Wire Wire Line
-	7800 1225 8100 1225
-Text Label 7800 1225 0    50   ~ 0
+	8100 1000 7800 1000
+Text Label 7800 1000 0    50   ~ 0
+Vsensor
+Wire Wire Line
+	7800 1100 8100 1100
+Text Label 7800 1100 0    50   ~ 0
+GND
+Wire Wire Line
+	7800 1200 8100 1200
+Text Label 7800 1200 0    50   ~ 0
 SCL
 Wire Wire Line
-	7800 1325 8100 1325
-Text Label 7800 1325 0    50   ~ 0
+	7800 1300 8100 1300
+Text Label 7800 1300 0    50   ~ 0
 SDA
 Wire Wire Line
-	7800 1425 8100 1425
-Text Label 7800 1425 0    50   ~ 0
+	7800 1400 8100 1400
+Text Label 7800 1400 0    50   ~ 0
 INT
 Wire Wire Line
@@
 	6975 5900 7425 5900
 Wire Wire Line
-	10250 1275 10550 1275
-Wire Wire Line
-	10250 1375 10550 1375
-Wire Wire Line
-	10250 1475 10550 1475
-Wire Wire Line
-	10250 1575 10550 1575
-Wire Wire Line
-	10250 1675 10550 1675
-Text Label 10250 1275 0    50   ~ 0
+	10200 1300 10500 1300
+Wire Wire Line
+	10200 1400 10500 1400
+Wire Wire Line
+	10200 1500 10500 1500
+Wire Wire Line
+	10200 1600 10500 1600
+Wire Wire Line
+	10200 1700 10500 1700
+Text Label 10200 1300 0    50   ~ 0
 VIN
-Text Label 10250 1375 0    50   ~ 0
-GND
-Text Label 10250 1575 0    50   ~ 0
+Text Label 10200 1400 0    50   ~ 0
+GND
+Text Label 10200 1600 0    50   ~ 0
 TX
-Text Label 10250 1675 0    50   ~ 0
+Text Label 10200 1700 0    50   ~ 0
 RX
 $Comp
 L Connector_Generic:Conn_01x05 J6
 U 1 1 60238DBA
-P 10750 1475
-F 0 "J6" H 10700 1775 50  0000 L CNN
-F 1 "Conn_01x05" H 10550 1175 50  0000 L CNN
-F 2 "Connector_PinHeader_2.54mm:PinHeader_1x05_P2.54mm_Vertical" H 10750 1475 50  0001 C CNN
-F 3 "~" H 10750 1475 50  0001 C CNN
-	1    10750 1475
+P 10700 1500
+F 0 "J6" H 10650 1800 50  0000 L CNN
+F 1 "Conn_01x05" H 10500 1200 50  0000 L CNN
+F 2 "Connector_PinHeader_2.54mm:PinHeader_1x05_P2.54mm_Vertical" H 10700 1500 50  0001 C CNN
+F 3 "~" H 10700 1500 50  0001 C CNN
+	1    10700 1500
 	1    0    0    -1
 $EndComp
 Text Notes 8800 1075 0    50   ~ 0
 Notes about Particule Meters sensors\n- PM_EN is optionnally intended to enable/disable the\nparticule meter (not to have it always on)
-Text Label 10250 1475 0    50   ~ 0
+Text Label 10200 1500 0    50   ~ 0
 PM_EN
 $Comp
@@
 L Connector_Generic:Conn_01x02 J2
 U 1 1 60D14B89
-P 5950 5550
-F 0 "J2" H 6030 5542 50  0000 L CNN
-F 1 "Conn_01x02" H 6030 5451 50  0000 L CNN
-F 2 "Connector_PinHeader_2.54mm:PinHeader_1x02_P2.54mm_Vertical" H 5950 5550 50  0001 C CNN
-F 3 "~" H 5950 5550 50  0001 C CNN
-	1    5950 5550
+P 5950 5650
+F 0 "J2" H 6030 5642 50  0000 L CNN
+F 1 "Conn_01x02" H 6030 5551 50  0000 L CNN
+F 2 "Connector_JST:JST_PH_S2B-PH-K_1x02_P2.00mm_Horizontal" H 5950 5650 50  0001 C CNN
+F 3 "~" H 5950 5650 50  0001 C CNN
+	1    5950 5650
 	1    0    0    -1
 $EndComp
@@
 Wire Notes Line
 	8550 4700 11150 4700
-Text Notes 6900 5000 0    50   ~ 0
+Text Notes 7200 5000 0    50   ~ 0
 USB power
 Text Notes 5750 5000 0    50   ~ 0
 Solar panel
 Wire Wire Line
+	5450 5750 5750 5750
+Text Label 5450 5750 0    50   ~ 0
+GND
+Wire Wire Line
 	5450 5650 5750 5650
 Text Label 5450 5650 0    50   ~ 0
-GND
-Wire Wire Line
-	5450 5550 5750 5550
-Text Label 5450 5550 0    50   ~ 0
 VS+
 Wire Wire Line
@@
 L Connector_Generic:Conn_01x05 J7
 U 1 1 60D63244
-P 7500 1225
-F 0 "J7" H 7450 1525 50  0000 L CNN
-F 1 "Conn_01x05" H 7300 925 50  0000 L CNN
-F 2 "Connector_PinHeader_2.54mm:PinHeader_1x05_P2.54mm_Vertical" H 7500 1225 50  0001 C CNN
-F 3 "~" H 7500 1225 50  0001 C CNN
-	1    7500 1225
-	1    0    0    -1
-$EndComp
-Wire Wire Line
-	7300 1025 7000 1025
-Text Label 7000 1025 0    50   ~ 0
-Vsensor
-Wire Wire Line
-	7000 1125 7300 1125
-Text Label 7000 1125 0    50   ~ 0
-GND
-Wire Wire Line
-	7000 1225 7300 1225
-Text Label 7000 1225 0    50   ~ 0
+P 7500 1200
+F 0 "J7" H 7450 1500 50  0000 L CNN
+F 1 "Conn_01x05" H 7300 900 50  0000 L CNN
+F 2 "Connector_PinHeader_2.54mm:PinHeader_1x05_P2.54mm_Vertical" H 7500 1200 50  0001 C CNN
+F 3 "~" H 7500 1200 50  0001 C CNN
+	1    7500 1200
+	1    0    0    -1
+$EndComp
+Wire Wire Line
+	7300 1000 7000 1000
+Text Label 7000 1000 0    50   ~ 0
+Vsensor
+Wire Wire Line
+	7000 1100 7300 1100
+Text Label 7000 1100 0    50   ~ 0
+GND
+Wire Wire Line
+	7000 1200 7300 1200
+Text Label 7000 1200 0    50   ~ 0
 SCL
 Wire Wire Line
-	7000 1325 7300 1325
-Text Label 7000 1325 0    50   ~ 0
+	7000 1300 7300 1300
+Text Label 7000 1300 0    50   ~ 0
 SDA
 Wire Wire Line
-	7000 1425 7300 1425
-Text Label 7000 1425 0    50   ~ 0
+	7000 1400 7300 1400
+Text Label 7000 1400 0    50   ~ 0
 INT
 Wire Wire Line
@@
 L Connector_Generic:Conn_01x04 J4
 U 1 1 60C16F38
-P 5575 1125
-F 0 "J4" H 5525 1325 50  0000 L CNN
-F 1 "Conn_01x04" H 5375 825 50  0000 L CNN
-F 2 "Connector_PinHeader_2.54mm:PinHeader_1x04_P2.54mm_Vertical" H 5575 1125 50  0001 C CNN
-F 3 "~" H 5575 1125 50  0001 C CNN
-	1    5575 1125
+P 5575 1100
+F 0 "J4" H 5525 1300 50  0000 L CNN
+F 1 "Conn_01x04" H 5375 800 50  0000 L CNN
+F 2 "Connector_PinHeader_2.54mm:PinHeader_1x04_P2.54mm_Vertical" H 5575 1100 50  0001 C CNN
+F 3 "~" H 5575 1100 50  0001 C CNN
+	1    5575 1100
 	1    0    0    -1
 $EndComp
@@
 L Connector_Generic:Conn_01x05 J3
 U 1 1 60E126AF
-P 6550 1225
-F 0 "J3" H 6500 1525 50  0000 L CNN
-F 1 "Conn_01x05" H 6325 925 50  0000 L CNN
-F 2 "Connector_PinHeader_2.54mm:PinHeader_1x05_P2.54mm_Vertical" H 6550 1225 50  0001 C CNN
-F 3 "~" H 6550 1225 50  0001 C CNN
-	1    6550 1225
-	1    0    0    -1
-$EndComp
-Wire Wire Line
-	6050 1425 6350 1425
-Text Label 6050 1425 0    50   ~ 0
+P 6550 1200
+F 0 "J3" H 6500 1500 50  0000 L CNN
+F 1 "Conn_01x05" H 6325 900 50  0000 L CNN
+F 2 "Connector_PinHeader_2.54mm:PinHeader_1x05_P2.54mm_Vertical" H 6550 1200 50  0001 C CNN
+F 3 "~" H 6550 1200 50  0001 C CNN
+	1    6550 1200
+	1    0    0    -1
+$EndComp
+Wire Wire Line
+	6050 1400 6350 1400
+Text Label 6050 1400 0    50   ~ 0
+INT
+Text Notes 5300 5450 0    50   ~ 0
+JST PH 2.0mm connector
+$Comp
+L Connector_Generic:Conn_01x05 J1
+U 1 1 60E0573E
+P 4650 1200
+F 0 "J1" H 4600 1500 50  0000 L CNN
+F 1 "Conn_01x05" H 4425 900 50  0000 L CNN
+F 2 "Connector_PinHeader_2.54mm:PinHeader_1x05_P2.54mm_Vertical" H 4650 1200 50  0001 C CNN
+F 3 "~" H 4650 1200 50  0001 C CNN
+	1    4650 1200
+	1    0    0    -1
+$EndComp
+Wire Wire Line
+	4150 1400 4450 1400
+Text Label 4150 1400 0    50   ~ 0
 INT
 $EndSCHEMATC
