File: pcb/lorawan-v2/neOsensor-LoRaWANV2.kicad_pcb (KiCad board)
At the start: 2 copper layers, 49.5 x 49.5 mm, 26 parts, among them J1 Conn_01x04, J2 Conn_01x02, J3 Conn_01x04, J4 Conn_01x05, J5 Conn_01x05, J6 Conn_01x05, J7 Conn_01x05, SW1 G71Y, U1 OLED1.3_I2C, U2 ATECC508A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

Commit message: lorawan-v2 pcb update
Parts:
- added R7: 47K, Resistor_SMD:R_0805_2012Metric_Pad1.15x1.40mm_HandSolder, B.Cu at (63.5, 46.2)
- added R8: 470, Resistor_SMD:R_0805_2012Metric_Pad1.15x1.40mm_HandSolder, F.Cu at (62.5, 45.2)
- added REF**: WEEE-Logo_4.2x6mm_SilkScreen, Symbol:WEEE-Logo_4.2x6mm_SilkScreen, F.Cu at (125.0, 57.7)
- added REF**: ESD-Logo_6.6x6mm_SilkScreen, Symbol:ESD-Logo_6.6x6mm_SilkScreen, F.Cu at (117.6, 57.1)
- added REF**: KiCad-Logo_8mm_SilkScreen, Symbol:KiCad-Logo_8mm_SilkScreen, F.Cu at (108.0, 68.6)
- added REF**: CE-Logo_8.5x6mm_SilkScreen, Symbol:CE-Logo_8.5x6mm_SilkScreen, F.Cu at (104.9, 55.4)
- added REF**: OSHW-Logo2_9.8x8mm_SilkScreen, Symbol:OSHW-Logo2_9.8x8mm_SilkScreen, F.Cu at (87.6, 38.4)
- C1, R3, U2: moved to B.Cu
- moved R1 67.3 mm to (76.0, 30.0), turned to 180 degrees
- moved R4 65.7 mm to (58.7, 34.8), turned to 180 degrees
- moved C1 64.6 mm to (72.9, 32.8), turned to 270 degrees
- moved R3 63.5 mm to (56.6, 34.8)
- moved C2 56.5 mm to (43.2, 64.8), turned to 270 degrees
- moved R2 49.1 mm to (73.9, 31.8), turned to 180 degrees
- moved R5 43.5 mm to (53.3, 65.0), turned to 90 degrees
- moved R6 43.1 mm to (63.5, 58.7), turned to 90 degrees
- moved U2 16.1 mm to (61.8, 68.1)
- moved JP1 1.48 mm to (45.7, 45.7)
- moved U3 1.46 mm to (48.0, 54.3)
- moved IR1 0.76 mm to (78.7, 55.9)
Routing:
- net /VIN: track 0.00 -> 14.9 mm, vias 0 -> 2
- net +3V3: track 0.00 -> 6.61 mm, vias 0 -> 23
- net /VDD: track 0.00 -> 3.02 mm
- net Net-(R1-Pad2): vias 0 -> 1
- net GND: vias 0 -> 16
- net /Vsensor: vias 0 -> 1
- net /SW1: vias 0 -> 1
- net /IR: vias 0 -> 1
- added copper zone on B.Cu, net +3V3
- added copper zone on F.Cu, net +3V3
Other:
- board text added: "(c)neO"
- board text added: "Campus"
- board text added: "CubeCell"
- board text added: "FT/jun21"
- board text added: "OLED"
- board text added: "RST / CLR"
- board text added: "RoHS"
- board text added: "Univ.Tlse3/IRIT"
- board text added: "neOSensor LoRaWAN V2"

Commit message: update
Parts:
- removed REF**: WEEE-Logo_4.2x6mm_SilkScreen, Symbol:WEEE-Logo_4.2x6mm_SilkScreen
- removed REF**: ESD-Logo_6.6x6mm_SilkScreen, Symbol:ESD-Logo_6.6x6mm_SilkScreen
- removed REF**: KiCad-Logo_8mm_SilkScreen, Symbol:KiCad-Logo_8mm_SilkScreen
- removed REF**: CE-Logo_8.5x6mm_SilkScreen, Symbol:CE-Logo_8.5x6mm_SilkScreen
- removed REF**: OSHW-Logo2_9.8x8mm_SilkScreen, Symbol:OSHW-Logo2_9.8x8mm_SilkScreen
- added C4: 100n, Capacitor_SMD:C_0805_2012Metric_Pad1.18x1.45mm_HandSolder, F.Cu at (70.2, 71.0)
- C3, J2, R4, R5: moved to B.Cu
- J4: value Conn_01x05 -> Conn_01x04; footprint Connector_PinHeader_2.54mm:PinHeader_1x05_P2.54mm_Vertical -> Connector_PinHeader_2.54mm:PinHeader_1x04_P2.54mm_Vertical
- J6, U3: moved to F.Cu
- moved J3 52.1 mm to (31.9, 36.2), turned to 0 degrees
- moved J5 43.3 mm to (59.6, 74.8), turned to 90 degrees
- moved J7 40.6 mm to (78.1, 54.6), turned to 0 degrees
- moved C3 30.5 mm to (48.5, 71.0), turned to 270 degrees
- moved JP1 22.4 mm to (35.9, 65.9)
- moved U3 20.3 mm to (39.1, 72.5), turned to 180 degrees
- moved IR1 11.7 mm to (78.7, 44.2)
- moved J2 9.67 mm to (43.2, 38.4), turned to 90 degrees
- moved J6 5.63 mm to (31.9, 61.8), turned to 0 degrees
- moved U2 5.10 mm to (66.9, 67.7), turned to 0 degrees
- moved R3 5.00 mm to (52.6, 37.7), turned to 180 degrees
- moved C2 3.59 mm to (43.6, 68.3), turned to 0 degrees
- moved R4 2.28 mm to (61.0, 34.8), turned to 90 degrees
- moved U1 1.53 mm to (55.0, 50.5)
- moved R5 1.03 mm to (52.3, 64.9), turned to 0 degrees
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Connections:
- U2 pad 1: Net-(U2-Pad1) -> (no net)
- U2 pad 2: Net-(U2-Pad2) -> (no net)
- U2 pad 3: Net-(U2-Pad3) -> (no net)
- U2 pad 7: Net-(U2-Pad7) -> (no net)
- U4 pad 11: Net-(U4-Pad11) -> (no net)
- U4 pad 12: Net-(U4-Pad12) -> (no net)
- U4 pad 15: Net-(U4-Pad15) -> (no net)
- U4 pad 18: Net-(U4-Pad18) -> (no net)
- U4 pad 19: Net-(U4-Pad19) -> (no net)
- U4 pad 20: Net-(U4-Pad20) -> (no net)
- U4 pad 4: Net-(U4-Pad4) -> (no net)
- U4 pad 8: Net-(U4-Pad8) -> (no net)
Routing:
- net /Vsensor: track 0.00 -> 206.0 mm, vias 1 -> 15
- net /SDA: track 0.00 -> 72.2 mm, vias 0 -> 3
- net /SCL: track 0.00 -> 68.7 mm, vias 0 -> 4
- net /VIN: track 14.9 -> 48.5 mm, vias 2 -> 1
- net /RX: track 0.00 -> 31.8 mm, vias 0 -> 1
- net /PM_EN: track 0.00 -> 31.8 mm
- net /VDD: track 3.02 -> 31.9 mm, vias 0 -> 2
- net /INT: track 0.00 -> 27.7 mm, vias 0 -> 1
- net /TX: track 0.00 -> 23.0 mm
- net /SW1: track 0.00 -> 18.8 mm, vias 1 -> 2
- net Net-(R5-Pad2): track 0.00 -> 3.18 mm, vias 0 -> 1
- net /VS+: track 0.00 -> 3.05 mm
- net +3V3: track 6.61 -> 9.47 mm, vias 23 -> 16
- added copper zone on B.Cu, net GND
- added copper zone on F.Cu, net GND
Other:
- board text added: "GND"
- board text added: "solar"

Commit message: neOSensor-LoRaWAN V2 ready for manfacturing
Parts:
- added REF**: ESD-Logo_6.6x6mm_SilkScreen, Symbol:ESD-Logo_6.6x6mm_SilkScreen, F.Cu at (50.2, 50.2)
- added REF**: CE-Logo_8.5x6mm_SilkScreen, Symbol:CE-Logo_8.5x6mm_SilkScreen, F.Cu at (71.4, 55.4)
- added REF**: KiCad-Logo2_5mm_SilkScreen, Symbol:KiCad-Logo2_5mm_SilkScreen, F.Cu at (68.5, 36.8)
- added REF**: OSHW-Logo2_9.8x8mm_SilkScreen, Symbol:OSHW-Logo2_9.8x8mm_SilkScreen, F.Cu at (66.0, 46.9)
- added REF**: RoHS-Logo_6mm_SilkScreen, Symbol:RoHS-Logo_6mm_SilkScreen, B.Cu at (51.8, 56.4)
- added REF**: WEEE-Logo_4.2x6mm_SilkScreen, Symbol:WEEE-Logo_4.2x6mm_SilkScreen, F.Cu at (43.6, 50.4)
- R7: moved to F.Cu
- moved R7 4.98 mm to (59.6, 49.3)
- moved R8 3.64 mm to (59.6, 47.4), turned to 180 degrees
- moved R2 0.63 mm to (73.9, 32.4)
- moved C1 0.51 mm to (72.9, 33.3)
- moved R1 0.51 mm to (76.0, 30.5)
- moved C2 0.38 mm to (43.6, 67.9)
Routing:
- net /SCL: track 68.7 -> 119.5 mm, vias 4 -> 8
- net /SDA: track 72.2 -> 117.6 mm, vias 3 -> 6
- net /IR: track 0.00 -> 25.4 mm, vias 1 -> 0
- net GND: track 0.00 -> 9.98 mm, vias 16 -> 26
- net Net-(R8-Pad1): track 0.00 -> 6.12 mm
- net Net-(R1-Pad2): track 0.00 -> 2.04 mm
- net /INT: track 27.7 -> 29.8 mm
Other:
- board text added: "Sensor LoRaWAN v2"
- board text added: "neO"
- board text removed: "RoHS"
- board text removed: "neOSensor LoRaWAN V2"

Commit message: update
Parts:
- removed REF**: ESD-Logo_6.6x6mm_SilkScreen, Symbol:ESD-Logo_6.6x6mm_SilkScreen
- removed REF**: CE-Logo_8.5x6mm_SilkScreen, Symbol:CE-Logo_8.5x6mm_SilkScreen
- removed REF**: KiCad-Logo2_5mm_SilkScreen, Symbol:KiCad-Logo2_5mm_SilkScreen
- removed REF**: OSHW-Logo2_9.8x8mm_SilkScreen, Symbol:OSHW-Logo2_9.8x8mm_SilkScreen
- removed REF**: RoHS-Logo_6mm_SilkScreen, Symbol:RoHS-Logo_6mm_SilkScreen
- removed REF**: WEEE-Logo_4.2x6mm_SilkScreen, Symbol:WEEE-Logo_4.2x6mm_SilkScreen
- C2: value 100nF -> 100n
- J3: value Conn_01x04 -> Conn_01x05; footprint Connector_PinHeader_2.54mm:PinHeader_1x04_P2.54mm_Vertical -> Connector_PinHeader_2.54mm:PinHeader_1x05_P2.54mm_Vertical
- moved J3 1.52 mm to (31.9, 34.7)
Connections:
- U4 pad 10: /SW1 -> /PM_EN
- U4 pad 13: /INT -> /SW1
- U4 pad 14: /PM_EN -> (no net)
- U4 pad 8: (no net) -> /INT

Commit message: update
Parts:
- J1: value Conn_01x04 -> Conn_01x05; footprint Connector_PinHeader_2.54mm:PinHeader_1x04_P2.54mm_Vertical -> Connector_PinHeader_2.54mm:PinHeader_1x05_P2.54mm_Vertical
- J2: footprint Connector_PinHeader_2.54mm:PinHeader_1x02_P2.54mm_Vertical -> Connector_JST:JST_PH_S2B-PH-K_1x02_P2.00mm_Horizontal
- R3, R4: moved to F.Cu
- moved R6 21.0 mm to (59.8, 38.0), turned to 0 degrees
- moved J4 15.2 mm to (55.9, 28.3)
- moved J1 4.95 mm to (50.7, 28.3), turned to 270 degrees
- moved R3 4.87 mm to (55.3, 33.7)
- moved R4 1.62 mm to (59.8, 33.7), turned to 0 degrees
- moved J2 1.17 mm to (43.9, 37.5)
Connections:
- U2 pad 1: (no net) -> Net-(U2-Pad1)
- U2 pad 2: (no net) -> Net-(U2-Pad2)
- U2 pad 3: (no net) -> Net-(U2-Pad3)
- U2 pad 7: (no net) -> Net-(U2-Pad7)
- U4 pad 11: (no net) -> Net-(U4-Pad11)
- U4 pad 12: (no net) -> Net-(U4-Pad12)
- U4 pad 14: (no net) -> Net-(U4-Pad14)
- U4 pad 15: (no net) -> Net-(U4-Pad15)
- U4 pad 18: (no net) -> Net-(U4-Pad18)
- U4 pad 19: (no net) -> Net-(U4-Pad19)
- U4 pad 20: (no net) -> Net-(U4-Pad20)
- U4 pad 4: (no net) -> Net-(U4-Pad4)
Routing:
- net /INT: track 29.8 -> 59.5 mm, vias 1 -> 3
- net /SDA: track 117.6 -> 100.1 mm, vias 6 -> 4
- net /Vsensor: track 205.7 -> 190.9 mm
- net /SCL: track 119.5 -> 104.9 mm, vias 8 -> 7
- net /SW1: track 18.8 -> 4.44 mm, vias 2 -> 1
- net /VS+: track 3.05 -> 4.25 mm
Other:
- board text added: "+"
- board text added: "Sensor LoRaWAN v2.1"
- board text removed: "GND"
- board text removed: "OLED"
- board text removed: "Sensor LoRaWAN v2"

Commit message: neOSensor LoRaWAN V2.1 pcb
Parts:
- added REF**: OSHW-Logo_7.5x8mm_SilkScreen, Symbol:OSHW-Logo_7.5x8mm_SilkScreen, B.Cu at (57.5, 67.6)
- added REF**: WEEE-Logo_4.2x6mm_SilkScreen, Symbol:WEEE-Logo_4.2x6mm_SilkScreen, B.Cu at (73.9, 52.5)
- added REF**: RoHS-Logo_6mm_SilkScreen, Symbol:RoHS-Logo_6mm_SilkScreen, B.Cu at (59.3, 57.3)
- added REF**: ESD-Logo_6.6x6mm_SilkScreen, Symbol:ESD-Logo_6.6x6mm_SilkScreen, B.Cu at (73.5, 61.6)
- added REF**: CE-Logo_8.5x6mm_SilkScreen, Symbol:CE-Logo_8.5x6mm_SilkScreen, B.Cu at (65.2, 48.4)
- added REF**: KiCad-Logo2_5mm_SilkScreen, Symbol:KiCad-Logo2_5mm_SilkScreen, B.Cu at (72.4, 37.0)
- moved J3 0.51 mm to (31.9, 35.2)
- moved R3 0.25 mm to (55.2, 33.4)
- moved R4 0.25 mm to (59.8, 33.4)
Routing:
- net /INT: track 59.5 -> 106.9 mm, vias 3 -> 5
- net /SW1: track 4.44 -> 38.0 mm, vias 1 -> 2
- net /PM_EN: track 31.8 -> 54.6 mm, vias 0 -> 1
- net /SCL: track 104.9 -> 123.7 mm, vias 7 -> 6
- net /SDA: track 100.1 -> 117.6 mm, vias 4 -> 5
- net /Vsensor: track 190.9 -> 201.5 mm
- net GND: track 9.98 -> 11.6 mm, vias 26 -> 29
Other:
- board text added: "1"
- board text added: "1,3" OLED 128 x 64"
- board text added: "3v3"
- board text added: "5v"
- board text added: "C L R"
- board text added: "Campus 2021"
- board text added: "CubeCell HTCC-AB01"
- board text added: "Dr THIEBOLT François original design"
- board text added: "GND"
- board text added: "INT"
- board text added: "IR"
- board text added: "If your computer performs ways slowly --> check nobody's asked for tea !! The hitchhicker's guide to the galaxy D.Adams 1952 - 2001"
- board text added: "PM_EN"
- board text added: "RX"
- board text added: "SCL"
- board text added: "SDA"
- board text added: "Serial"
- board text added: "TX"
- board text added: "Univ-tlse3/IRIT"
- board text added: "Universities are GREAT !"
- board text added: "VS+"
- board text added: "https://github.com/fthiebolt/neOCampus-arduino"
- board text removed: "Campus"
- board text removed: "CubeCell"
- board text removed: "RST / CLR"
- board text removed: "Univ.Tlse3/IRIT"
