File: pcb/neOClock/neOClock.kicad_pcb (KiCad board)
At the start: 2 copper layers, 23 parts, among them J1 Barrel_Jack, J2 Conn_01x04, J3 Conn_01x04, J4 Conn_01x04, SW1 SW_Push, SW2 SW_Push, SW3 SW_Push, U1 MAX6959AAEE+, U10 KCSC02-136, U11 KCSC02-136, U12 YAAJ_DCDC_StepDown_LM2596, U13 AMS1117, U2 KCSC02-136, U3 ESP32_dev_30p, U9 KCSC02-136

Commit message: update
Parts:
- removed D8: LED, LED_THT:LED_D5.0mm
- removed U10, U11, U9: KCSC02-136, Display_7Segment:SA15-11xxx
- removed U12: YAAJ_DCDC_StepDown_LM2596, DC-DC_LM2596:DC_DC_LM2596
- removed U13: AMS1117, Package_TO_SOT_SMD:SOT-223-3_TabPin2
- added C4: 470µF, Capacitor_THT:CP_Radial_D5.0mm_P2.50mm, F.Cu at (62.0, 190.5)
- added D2: APA102, LED_SMD:LED_RGB_5050-6, F.Cu at (68.7, 178.2)
- added D3: APA102, LED_SMD:LED_RGB_5050-6, F.Cu at (51.6, 178.5)
- added D4: APA102, LED_SMD:LED_RGB_5050-6, F.Cu at (60.4, 178.2)
- added J5: 78_01_030_0004, neosensor_addon:HARTING_78_01_030_0004, F.Cu at (40.0, 137.4)
- added Q1: Q_NPN_CBE, Package_TO_SOT_SMD:SC-59_Handsoldering, F.Cu at (29.7, 188.5)
- added Q2: Q_NPN_CBE, Package_TO_SOT_SMD:SC-59_Handsoldering, F.Cu at (36.4, 188.5)
- added U4: HDSP-7801, Display_7Segment:SBC18-11SURKCGKWA, F.Cu at (142.1, 67.7)
- added U5: HDSP-7801, Display_7Segment:SBC18-11SURKCGKWA, F.Cu at (263.9, 67.6)
- added U6: SAA1064, neosensor_addon:SAA1064, F.Cu at (67.6, 132.5)
- added U7: HDSP-7801, Display_7Segment:SBC18-11SURKCGKWA, F.Cu at (183.8, 67.7)
- added U8: HDSP-7801, Display_7Segment:SBC18-11SURKCGKWA, F.Cu at (224.5, 67.7)
- D5: value LED -> APA102; footprint LED_THT:LED_D5.0mm -> LED_SMD:LED_RGB_5050-6
- SW1, SW2, SW3: footprint Button_Switch_SMD:SW_Push_1P1T_NO_CK_KMR2 -> Button_Switch_SMD:SW_Push_1P1T_NO_6x6mm_H9.5mm
- U1: value MAX6959AAEE+ -> YAAJ_DCDC_StepDown_LM2596; footprint max6959:MAX6959AAEE&plus_ -> neosensor_addon:DC_DC_LM2596
- U2: value KCSC02-136 -> AMS1117; footprint Display_7Segment:SA15-11xxx -> Package_TO_SOT_SMD:SOT-223-3_TabPin2
- moved SW1 227.8 mm to (132.7, 191.3)
- moved SW2 218.9 mm to (140.1, 181.7)
- moved SW3 214.4 mm to (128.9, 181.6)
- moved J3 212.3 mm to (99.8, 184.8)
- moved J2 212.2 mm to (93.7, 185.5)
- moved J4 208.5 mm to (88.8, 186.3)
- moved D6 200.6 mm to (73.2, 190.5)
- moved U3 197.9 mm to (29.2, 64.6)
- moved D5 182.1 mm to (79.4, 177.8)
- moved D7 179.4 mm to (81.4, 190.4)
- moved J1 150.2 mm to (113.4, 185.5)
- moved D1 139.5 mm to (44.8, 186.6)
- moved U1 130.3 mm to (57.9, 34.2), turned to 180 degrees
- moved C1 73.5 mm to (52.6, 190.2)
- moved C2 71.5 mm to (44.7, 192.3)
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Connections:
- net Net-(SW2-Pad2) renamed Push_2
- C1 pad 1: /Alim/5v -> 5v
- C2 pad 1: /Alim/3v3 -> 3v3
- D1 pad 2: Net-(D1-Pad2) -> 12v
- D5 pad 1: Net-(D5-Pad1) -> Net-(D4-Pad6)
- D5 pad 2: Net-(D5-Pad2) -> Net-(D4-Pad5)
- D6 pad 1: Net-(D6-Pad1) -> 0
- D7 pad 1: Net-(D5-Pad2) -> 0
- D7 pad 2: Net-(D5-Pad1) -> Net-(D7-Pad2)
- IR1 pad 1: /Alim/3v3 -> 3v3
- IR1 pad 2: Net-(IR1-Pad2) -> IR
- J2 pad 1: /digit/Scl -> 3v3
- J2 pad 2: /digit/Sda -> SDA
- J2 pad 3: /Alim/3v3 -> SCL
- J3 pad 1: /digit/Scl -> 3v3
- J3 pad 2: /digit/Sda -> SDA
- J3 pad 3: /Alim/3v3 -> SCL
- J4 pad 1: /digit/Scl -> 3v3
- J4 pad 2: /digit/Sda -> SDA
- J4 pad 3: /Alim/3v3 -> SCL
- SW1 pad 1: /Alim/3v3 -> 3v3
- SW1 pad 2: Net-(SW1-Pad2) -> Push_1
- SW2 pad 1: /Alim/3v3 -> 3v3
- SW3 pad 1: /Alim/3v3 -> 3v3
- SW3 pad 2: Net-(SW3-Pad2) -> Push_3
- U1 pad 1: /digit/Sda -> 12v
- U1 pad 2: /digit/Scl -> 0
- U1 pad 3: Net-(U1-Pad3) -> 0
- U1 pad 4: Net-(D5-Pad1) -> 5v
- U2 pad 1: Net-(U1-Pad11) -> 0
- U2 pad 2: Net-(U1-Pad12) -> 3v3
- U2 pad 3: Net-(D5-Pad1) -> 5v
- U3 pad 10: Net-(IR1-Pad2) -> Net-(U3-Pad10)
- U3 pad 11: /digit/Sda -> SDA
- U3 pad 12: /digit/Input1 -> CI
- U3 pad 13: /digit/Input2 -> DI
- U3 pad 14: /digit/Scl -> SCL
- U3 pad 17: Net-(SW3-Pad2) -> Push_1
- U3 pad 19: Net-(SW1-Pad2) -> Push_3
- U3 pad 20: Net-(U3-Pad20) -> IR
- U3 pad 30: /Alim/5v -> 5v

Commit message: update
Parts:
- D1: value DIODE -> LED; footprint Diode_SMD:D_0603_1608Metric_Pad1.05x0.95mm_HandSolder -> LED_THT:LED_D5.0mm
- J5: footprint neosensor_addon:HARTING_78_01_030_0004 -> neosensor_addon:ATECC508A
- Q1: value Q_NPN_CBE -> BC337
- moved D6 169.3 mm to (67.2, 21.3)
- moved D7 169.1 mm to (85.1, 21.3)
- moved D1 168.1 mm to (75.7, 21.3)
- moved J5 76.8 mm to (52.5, 61.6)
- moved U6 59.9 mm to (91.7, 77.6)
Connections:
- D1 pad 1: Net-(D1-Pad1) -> 12v
- D1 pad 2: 12v -> Net-(D1-Pad2)
- J1 pad 1: Net-(D1-Pad1) -> Net-(D1-Pad2)

Commit message: update
Parts:
- added D10: APA102, LED_SMD:LED_RGB_5050-6, F.Cu at (187.7, 224.4)
- added D11: APA102, LED_SMD:LED_RGB_5050-6, F.Cu at (179.3, 237.5)
- added D12: APA102, LED_SMD:LED_RGB_5050-6, F.Cu at (187.7, 230.9)
- added D13: APA102, LED_SMD:LED_RGB_5050-6, F.Cu at (196.0, 224.4)
- added D14: APA102, LED_SMD:LED_RGB_5050-6, F.Cu at (187.7, 237.5)
- added D15: APA102, LED_SMD:LED_RGB_5050-6, F.Cu at (196.0, 230.9)
- added D8: APA102, LED_SMD:LED_RGB_5050-6, F.Cu at (179.3, 224.4)
- added D9: APA102, LED_SMD:LED_RGB_5050-6, F.Cu at (179.3, 230.9)
- added H1: MountingHole_Pad, MountingHole:MountingHole_3.2mm_M3_Pad, F.Cu at (144.0, 74.2)
- added H2: MountingHole_Pad, MountingHole:MountingHole_3.2mm_M3_Pad, F.Cu at (167.0, 77.6)
- added H3: MountingHole_Pad, MountingHole:MountingHole_3.2mm_M3_Pad, F.Cu at (144.0, 82.2)
- added H4: MountingHole_Pad, MountingHole:MountingHole_3.2mm_M3_Pad, F.Cu at (158.5, 87.6)
- J5: value 78_01_030_0004 -> ATECC508A
- SW1, SW2, SW3: value SW_Push -> G71Y; footprint Button_Switch_SMD:SW_Push_1P1T_NO_6x6mm_H9.5mm -> neosensor_addon:G71Y_µsw_smd
- U1: value YAAJ_DCDC_StepDown_LM2596 -> DCDC_LM2596
- moved J5 244.6 mm to (292.4, 14.1)
- moved U6 220.0 mm to (305.7, 26.5)
- moved U8 205.7 mm to (22.5, 29.1), turned to 0 degrees
- moved Q2 189.6 mm to (225.1, 206.9)
- moved U5 187.0 mm to (80.9, 29.1), turned to 0 degrees
- moved U3 181.3 mm to (208.8, 39.4)
- moved C1 176.7 mm to (225.6, 226.3)
- moved Q1 162.7 mm to (190.2, 215.2)
- moved U7 160.9 mm to (22.9, 69.1), turned to 0 degrees
- moved D3 160.4 mm to (209.2, 207.9)
- moved D4 160.0 mm to (217.6, 207.9)
- moved C4 149.6 mm to (208.9, 218.6)
- moved U2 148.5 mm to (197.1, 71.8)
- moved D2 135.5 mm to (200.9, 207.9)
- moved J1 128.7 mm to (239.3, 212.6)
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Connections:
- SW1 pad 1: 3v3 -> Push_1
- SW1 pad 2: Push_1 -> Net-(SW1-Pad2)
- SW2 pad 1: 3v3 -> Push_2
- SW2 pad 2: Push_2 -> Net-(SW2-Pad2)
- SW3 pad 1: 3v3 -> Push_3
- SW3 pad 2: Push_3 -> Net-(SW3-Pad2)

Commit message: mise a jour des schema
Parts:
- added H5: MountingHole_Pad, MountingHole:MountingHole_3.2mm_M3_Pad, F.Cu at (18.6, 78.9)
- added H6: MountingHole_Pad, MountingHole:MountingHole_3.2mm_M3_Pad, F.Cu at (196.2, 29.4)
- C1, C2, C4, D1, D10, D11, D12, D13, D14, D15, D2, D3, D4, D5, D8, D9, J1, J2, J3, J4, Q1, Q2, SW1, SW2, SW3, U1, U2, U3: moved to B.Cu
- J5: footprint neosensor_addon:ATECC508A -> neosensor_addon:SOIC-8_3.9x5.4mm_P1.27mm_HandSolder
- U6: footprint neosensor_addon:SAA1064 -> neosensor_addon:SOIC-24W_7.5x15.4mm_P1.27mm_HandSolder
- moved U6 310.2 mm to (-2.96, 57.1)
- moved J5 281.3 mm to (11.8, 34.5)
- moved D2 250.1 mm to (26.2, 29.0), turned to 180 degrees
- moved D15 243.0 mm to (61.0, 29.0), turned to 180 degrees
- moved D14 227.9 mm to (95.8, 29.0), turned to 180 degrees
- moved D3 223.7 mm to (26.1, 79.3)
- moved Q2 210.9 mm to (95.0, 40.9)
- moved D13 210.0 mm to (119.0, 29.0), turned to 180 degrees
- moved D11 208.7 mm to (188.6, 29.0), turned to 180 degrees
- moved D12 204.8 mm to (153.8, 29.0), turned to 180 degrees
- moved D4 202.6 mm to (61.0, 79.3)
- moved J2 198.3 mm to (31.4, 81.0), turned to 270 degrees
- moved J4 185.3 mm to (40.5, 81.0), turned to 270 degrees
- moved J3 181.6 mm to (49.6, 81.0), turned to 270 degrees
- moved C1 180.9 mm to (173.5, 53.0)
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Connections:
- U7 pad 10: Net-(U6-PadP9) -> Net-(U7-Pad10)
- U7 pad 2: Net-(U6-PadP14) -> Net-(U7-Pad2)
- U7 pad 3: Net-(U6-PadP15) -> Net-(U7-Pad3)
- U7 pad 4: Net-(U6-PadP13) -> Net-(U7-Pad4)
- U7 pad 5: Net-(U6-PadP12) -> Net-(U7-Pad5)
- U7 pad 7: Net-(U6-PadP16) -> Net-(U7-Pad7)
- U7 pad 8: Net-(U6-PadP11) -> Net-(U7-Pad8)
- U7 pad 9: Net-(U6-PadP10) -> Net-(U7-Pad9)
- U8 pad 10: Net-(U6-PadP9) -> Net-(U7-Pad10)
- U8 pad 2: Net-(U6-PadP14) -> Net-(U7-Pad2)
- U8 pad 3: Net-(U6-PadP15) -> Net-(U7-Pad3)
- U8 pad 4: Net-(U6-PadP13) -> Net-(U7-Pad4)
- U8 pad 5: Net-(U6-PadP12) -> Net-(U7-Pad5)
- U8 pad 7: Net-(U6-PadP16) -> Net-(U7-Pad7)
- U8 pad 8: Net-(U6-PadP11) -> Net-(U7-Pad8)
- U8 pad 9: Net-(U6-PadP10) -> Net-(U7-Pad9)
Routing:
- net Net-(Q1-Pad3): track 0.00 -> 217.8 mm, vias 0 -> 9
- net Net-(Q2-Pad3): track 0.00 -> 214.2 mm, vias 0 -> 7
- net 5v: track 0.00 -> 179.2 mm, vias 0 -> 4
- net 12v: track 0.00 -> 134.8 mm, vias 0 -> 5
- net Net-(U4-Pad7): track 0.00 -> 110.6 mm, vias 0 -> 4
- net Net-(U7-Pad5): track 0.00 -> 108.1 mm, vias 0 -> 4
- net Net-(U7-Pad4): track 0.00 -> 103.8 mm, vias 0 -> 4
- net Net-(U4-Pad5): track 0.00 -> 102.6 mm, vias 0 -> 4
- net Net-(U4-Pad8): track 0.00 -> 99.1 mm, vias 0 -> 4
- net Net-(U4-Pad9): track 0.00 -> 98.2 mm, vias 0 -> 4
- net Net-(U7-Pad3): track 0.00 -> 97.8 mm, vias 0 -> 4
- net Net-(U7-Pad2): track 0.00 -> 97.6 mm, vias 0 -> 4
- net Net-(U4-Pad10): track 0.00 -> 96.5 mm, vias 0 -> 4
- net Net-(U7-Pad10): track 0.00 -> 94.8 mm, vias 0 -> 3
- net Net-(U4-Pad3): track 0.00 -> 94.0 mm, vias 0 -> 4
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- added copper zone on B.Cu, net 0
- added copper zone on F.Cu, net 0
Other:
- board outline added: 200 x 139.5 mm

Commit message: update
Parts:
- removed D6, D7: LED, LED_THT:LED_D5.0mm
- removed H5, H6: MountingHole_Pad, MountingHole:MountingHole_3.2mm_M3_Pad
- added C3: 1µF, Resistor_SMD:R_0805_2012Metric_Pad1.20x1.40mm_HandSolder, F.Cu at (109.3, 39.7)
- added C5: 100µF, Capacitor_THT:CP_Radial_D5.0mm_P2.50mm, F.Cu at (221.3, -46.4)
- added R1: 15k, Resistor_SMD:R_0805_2012Metric_Pad1.20x1.40mm_HandSolder, F.Cu at (99.8, 39.7)
- added R2: 15K, Resistor_SMD:R_0805_2012Metric_Pad1.20x1.40mm_HandSolder, F.Cu at (213.2, -38.7)
- added R3: 15K, Resistor_SMD:R_0805_2012Metric_Pad1.20x1.40mm_HandSolder, F.Cu at (183.7, 22.0)
- added R4: 15K, Resistor_SMD:R_0805_2012Metric_Pad1.20x1.40mm_HandSolder, F.Cu at (213.2, -35.8)
- added R5: 15K, Resistor_SMD:R_0805_2012Metric_Pad1.20x1.40mm_HandSolder, F.Cu at (228.2, -48.2)
- added R6: 15K, Resistor_SMD:R_0805_2012Metric_Pad1.20x1.40mm_HandSolder, F.Cu at (204.9, -27.2)
- added R7: 15K, Resistor_SMD:R_0805_2012Metric_Pad1.20x1.40mm_HandSolder, F.Cu at (204.9, -24.2)
- added R8: 4.7K, Resistor_SMD:R_0805_2012Metric_Pad1.20x1.40mm_HandSolder, F.Cu at (212.8, -32.8)
- added R9: 4.7K, Resistor_SMD:R_0805_2012Metric_Pad1.20x1.40mm_HandSolder, F.Cu at (70.4, 36.9)
- C1: value 470µF -> 1µF; footprint Capacitor_THT:CP_Radial_D5.0mm_P2.50mm -> Resistor_SMD:R_0805_2012Metric_Pad1.20x1.40mm_HandSolder; moved to F.Cu
- C2: value 100µF -> 1µF; footprint Capacitor_Tantalum_SMD:CP_EIA-3216-18_Kemet-A_Pad1.58x1.35mm_HandSolder -> Resistor_SMD:R_0805_2012Metric_Pad1.20x1.40mm_HandSolder; moved to F.Cu
- C4: value 470µF -> 100nF; footprint Capacitor_THT:CP_Radial_D5.0mm_P2.50mm -> Resistor_SMD:R_0805_2012Metric_Pad1.20x1.40mm_HandSolder; moved to F.Cu
- D1: value LED -> 1N4148; footprint LED_THT:LED_D5.0mm -> Diode_THT:D_DO-35_SOD27_P7.62mm_Horizontal; moved to F.Cu
- D10, D11, D12, D13, D14, D15, D2, D3, D4, D5, D8, D9, J2, J3, J4, SW1, SW2, SW3, U1, U2, U3: moved to F.Cu
- J1: footprint Connector_BarrelJack:BarrelJack_CUI_PJ-036AH-SMT_Horizontal -> Connector_BarrelJack:BarrelJack_Horizontal; moved to F.Cu
- Q1: value BC337 -> 2n2222a; moved to F.Cu
- Q2: value Q_NPN_CBE -> 2n2222a; footprint Package_TO_SOT_SMD:SC-59_Handsoldering -> Package_TO_SOT_THT:TO-92; moved to F.Cu
- moved H1 215.2 mm to (222.6, -39.2)
- moved D2 203.4 mm to (215.0, -46.4), turned to 0 degrees
- moved H4 197.6 mm to (206.5, -32.6)
- moved D4 192.5 mm to (206.7, -46.4)
- moved D5 178.1 mm to (215.0, -53.0)
- moved U3 166.4 mm to (187.7, -30.4), turned to 0 degrees
- moved D3 160.9 mm to (177.1, 23.8)
- moved U8 160.1 mm to (62.2, -41.6), turned to 0 degrees
- moved D8 158.7 mm to (206.7, -53.0)
- moved D13 132.7 mm to (223.4, -53.0), turned to 0 degrees
- moved U5 127.9 mm to (120.0, -41.6), turned to 0 degrees
- moved J5 126.3 mm to (137.8, 26.1)
- moved J1 123.6 mm to (71.8, 28.2), turned to 0 degrees
- moved D1 118.4 mm to (58.9, 37.2)
- moved U4 116.0 mm to (120.0, -2.02), turned to 0 degrees
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Connections:
- C1 pad 1: 5v -> Push_1
- C2 pad 1: 3v3 -> Push_2
- C4 pad 1: 12v -> 5v
- D10 pad 4: 3v3 -> 5v
- D11 pad 4: 3v3 -> 5v
- D12 pad 4: 3v3 -> 5v
- D13 pad 4: 3v3 -> 5v
- D14 pad 4: 3v3 -> 5v
- D15 pad 4: 3v3 -> 5v
- D2 pad 4: 3v3 -> 5v
- D3 pad 4: 3v3 -> 5v
- D4 pad 4: 3v3 -> 5v
- D5 pad 4: 3v3 -> 5v
- D8 pad 4: 3v3 -> 5v
- D9 pad 4: 3v3 -> 5v
- Q1 pad 2: Net-(Q1-Pad2) -> /a1
- Q2 pad 2: Net-(Q2-Pad2) -> /b1
- SW1 pad 1: Push_1 -> Net-(R2-Pad1)
- SW1 pad 2: Net-(SW1-Pad2) -> 3v3
- SW1 pad 3: Net-(SW1-Pad2) -> 0
- SW2 pad 1: Push_2 -> Net-(R3-Pad1)
- SW2 pad 2: Net-(SW2-Pad2) -> 3v3
- SW2 pad 3: Net-(SW2-Pad2) -> 0
- SW3 pad 1: Push_3 -> Net-(R4-Pad1)
- SW3 pad 2: Net-(SW3-Pad2) -> 3v3
- SW3 pad 3: Net-(SW3-Pad2) -> 0
- U3 pad 12: CI -> Net-(U3-Pad12)
- U3 pad 13: DI -> Net-(U3-Pad13)
- U3 pad 15: Net-(U3-Pad15) -> DI
- U3 pad 20: IR -> Net-(U3-Pad20)
- U3 pad 5: Net-(U3-Pad5) -> IR
- U3 pad 9: Net-(U3-Pad9) -> CI
- U4 pad 10: Net-(U4-Pad10) -> /a10
- U4 pad 2: Net-(U4-Pad2) -> /a2
- U4 pad 3: Net-(U4-Pad3) -> /a3
- U4 pad 4: Net-(U4-Pad4) -> /a4
- U4 pad 5: Net-(U4-Pad5) -> /a5
- U4 pad 7: Net-(U4-Pad7) -> /a7
- U4 pad 8: Net-(U4-Pad8) -> /a8
- U4 pad 9: Net-(U4-Pad9) -> /a9
- U5 pad 10: Net-(U4-Pad10) -> /a10
- U5 pad 2: Net-(U4-Pad2) -> /a2
- U5 pad 3: Net-(U4-Pad3) -> /a3
- U5 pad 4: Net-(U4-Pad4) -> /a4
- U5 pad 5: Net-(U4-Pad5) -> /a5
- U5 pad 7: Net-(U4-Pad7) -> /a7
- U5 pad 8: Net-(U4-Pad8) -> /a8
- U5 pad 9: Net-(U4-Pad9) -> /a9
- U6 pad 1: Net-(U6-Pad1) -> 0
- U6 pad 10: Net-(U6-Pad10) -> /a10
- U6 pad 11: Net-(U6-Pad11) -> /a1
- U6 pad 12: Net-(U6-Pad12) -> 0
- U6 pad 13: Net-(U6-Pad13) -> 12v
- U6 pad 14: Net-(U6-Pad14) -> /b1
- U6 pad 15: Net-(U6-Pad15) -> /b10
- U6 pad 16: Net-(U6-Pad16) -> /b9
- U6 pad 17: Net-(U6-Pad17) -> /b8
- U6 pad 18: Net-(U6-Pad18) -> /b5
- U6 pad 19: Net-(U6-Pad19) -> /b4
- U6 pad 2: Net-(U6-Pad2) -> 0
- U6 pad 20: Net-(U6-Pad20) -> /b2
- U6 pad 21: Net-(U6-Pad21) -> /b3
- U6 pad 22: Net-(U6-Pad22) -> /b7
- U6 pad 23: Net-(U6-Pad23) -> SDA
- U6 pad 24: Net-(U6-Pad24) -> SCL
- U6 pad 3: Net-(U6-Pad3) -> /a7
- U6 pad 4: Net-(U6-Pad4) -> /a3
- U6 pad 5: Net-(U6-Pad5) -> /a2
- U6 pad 6: Net-(U6-Pad6) -> /a4
- U6 pad 7: Net-(U6-Pad7) -> /a5
- U6 pad 8: Net-(U6-Pad8) -> /a8
- U6 pad 9: Net-(U6-Pad9) -> /a9
- U7 pad 10: Net-(U7-Pad10) -> /b10
- U7 pad 2: Net-(U7-Pad2) -> /b2
- U7 pad 3: Net-(U7-Pad3) -> /b3
- U7 pad 4: Net-(U7-Pad4) -> /b4
- U7 pad 5: Net-(U7-Pad5) -> /b5
- U7 pad 7: Net-(U7-Pad7) -> /b7
- U7 pad 8: Net-(U7-Pad8) -> /b8
- U7 pad 9: Net-(U7-Pad9) -> /b9
- U8 pad 10: Net-(U7-Pad10) -> /b10
- U8 pad 2: Net-(U7-Pad2) -> /b2
- U8 pad 3: Net-(U7-Pad3) -> /b3
- U8 pad 4: Net-(U7-Pad4) -> /b4
- U8 pad 5: Net-(U7-Pad5) -> /b5
- U8 pad 7: Net-(U7-Pad7) -> /b7
- U8 pad 8: Net-(U7-Pad8) -> /b8
- U8 pad 9: Net-(U7-Pad9) -> /b9
Routing:
- net Net-(Q1-Pad3): track 217.8 -> 0.00 mm, vias 9 -> 0
- net Net-(Q2-Pad3): track 214.2 -> 0.00 mm, vias 7 -> 0
- net 5v: track 179.2 -> 0.00 mm, vias 4 -> 0
- net 12v: track 134.8 -> 0.00 mm, vias 5 -> 0
- net Net-(U4-Pad7): track 110.6 -> 0.00 mm, vias 4 -> 0
- net Net-(U7-Pad5): track 108.1 -> 0.00 mm, vias 4 -> 0
- net Net-(U7-Pad4): track 103.8 -> 0.00 mm, vias 4 -> 0
- net Net-(U4-Pad5): track 102.6 -> 0.00 mm, vias 4 -> 0
- net Net-(U4-Pad8): track 99.1 -> 0.00 mm, vias 4 -> 0
- net Net-(U4-Pad9): track 98.2 -> 0.00 mm, vias 4 -> 0
- net Net-(U7-Pad3): track 97.8 -> 0.00 mm, vias 4 -> 0
- net Net-(U7-Pad2): track 97.6 -> 0.00 mm, vias 4 -> 0
- net Net-(U4-Pad10): track 96.5 -> 0.00 mm, vias 4 -> 0
- net Net-(U7-Pad10): track 94.8 -> 0.00 mm, vias 3 -> 0
- net Net-(U4-Pad3): track 94.0 -> 0.00 mm, vias 4 -> 0
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- removed copper zone on B.Cu, net 0
- removed copper zone on F.Cu, net 0
Other:
- board size 200 x 139.5 mm -> 200 x 80 mm

Commit message: update
Parts:
- C1, C2, C3, C4, C5, D1, D10, D11, D12, D13, D14, D15, D2, D3, D4, D5, D8, D9, J1, J5, Q2, R1, R2, R3, R4, R5, R6, R7, R8, R9, SW1, SW2, SW3, U1, U2, U3, U6: moved to B.Cu
- Q1: footprint Package_TO_SOT_SMD:SC-59_Handsoldering -> Package_TO_SOT_THT:TO-92; moved to B.Cu
- U4, U5, U7, U8: value HDSP-7801 -> SA15-11GWA; footprint Display_7Segment:SBC18-11SURKCGKWA -> Display_7Segment:SA15-11xxx
- moved D2 206.6 mm to (18.7, 17.8), turned to 180 degrees
- moved D4 198.4 mm to (64.7, 92.2)
- moved C2 186.3 mm to (38.7, 23.6)
- moved R5 184.7 mm to (57.0, 21.2), turned to 180 degrees
- moved D5 183.2 mm to (103.3, 92.2)
- moved R4 179.8 mm to (42.7, 21.2), turned to 180 degrees
- moved R6 175.0 mm to (36.7, 21.2), turned to 180 degrees
- moved H4 174.0 mm to (43.3, 27.9)
- moved D3 172.6 mm to (18.7, 92.2)
- moved R2 171.2 mm to (52.9, 21.1), turned to 180 degrees
- moved R8 171.0 mm to (57.7, 39.2), turned to 180 degrees
- moved U3 168.8 mm to (42.2, 55.0), turned to 90 degrees
- moved D8 165.8 mm to (126.7, 92.2)
- moved R7 164.4 mm to (46.8, 21.2), turned to 180 degrees
- moved U8 153.4 mm to (161.4, 75.4), turned to 90 degrees
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Connections:
- net /a1 renamed /a1_5
- net /b1 renamed /b1_5
- U4 pad 5: /a5 -> Net-(Q1-Pad3)
- U4 pad 6: Net-(Q1-Pad3) -> /a6
- U5 pad 5: /a5 -> Net-(Q2-Pad3)
- U5 pad 6: Net-(Q2-Pad3) -> /a6
- U6 pad 10: /a10 -> /a7
- U6 pad 15: /b10 -> /b7
- U6 pad 16: /b9 -> /b6
- U6 pad 17: /b8 -> /b4
- U6 pad 18: /b5 -> /b3
- U6 pad 19: /b4 -> /b2
- U6 pad 20: /b2 -> /b9
- U6 pad 21: /b3 -> /b10
- U6 pad 22: /b7 -> /b8
- U6 pad 3: /a7 -> /a8
- U6 pad 4: /a3 -> /a10
- U6 pad 5: /a2 -> /a9
- U6 pad 6: /a4 -> /a2
- U6 pad 7: /a5 -> /a3
- U6 pad 8: /a8 -> /a4
- U6 pad 9: /a9 -> /a6
- U7 pad 2: /b2 -> /b4
- U7 pad 3: /b3 -> /b7
- U7 pad 4: /b4 -> /b2
- U7 pad 5: /b5 -> Net-(Q1-Pad3)
- U7 pad 6: Net-(Q1-Pad3) -> /b9
- U7 pad 7: /b7 -> /b3
- U7 pad 9: /b9 -> /b6
- U8 pad 5: /b5 -> Net-(Q2-Pad3)
- U8 pad 6: Net-(Q2-Pad3) -> /b6
Routing:
- net /b6: track 0.00 -> 142.8 mm, vias 0 -> 4
- net /b9: track 0.00 -> 131.3 mm, vias 0 -> 4
- net /b8: track 0.00 -> 129.7 mm, vias 0 -> 4
- net Net-(Q1-Pad3): track 0.00 -> 128.4 mm, vias 0 -> 6
- net /b10: track 0.00 -> 119.3 mm, vias 0 -> 4
- net /b3: track 0.00 -> 107.2 mm, vias 0 -> 5
- net /b4: track 0.00 -> 106.3 mm, vias 0 -> 3
- net /a8: track 0.00 -> 94.4 mm, vias 0 -> 4
- net Net-(Q2-Pad3): track 0.00 -> 92.8 mm, vias 0 -> 6
- net /b2: track 0.00 -> 92.6 mm, vias 0 -> 4
- net /a10: track 0.00 -> 92.0 mm, vias 0 -> 4
- net /a9: track 0.00 -> 91.9 mm, vias 0 -> 4
- net /a6: track 0.00 -> 87.6 mm, vias 0 -> 4
- net /a7: track 0.00 -> 85.8 mm, vias 0 -> 4
- net /b7: track 0.00 -> 75.6 mm, vias 0 -> 3
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- added copper zone on B.Cu, net 0
- added copper zone on F.Cu, net 0
Other:
- net class power added: clearance 0.2, trace_width 0.66, via_dia 1.2, via_drill 0.6

Commit message: update
Parts:
- removed D10, D11, D12, D13, D14, D15, D2: APA102, LED_SMD:LED_RGB_5050-6
- D3, D4, D5, D8, D9: footprint LED_SMD:LED_RGB_5050-6 -> LED_SMD:LED_WS2812_PLCC6_5.0x5.0mm_P1.6mm
- moved J2 124.0 mm to (77.0, 93.4)
- moved J3 124.0 mm to (67.7, 93.4)
- moved J4 124.0 mm to (58.4, 93.4)
- moved D9 87.6 mm to (211.3, 17.9)
- moved D8 83.6 mm to (165.0, 17.9)
- moved D5 75.2 mm to (115.0, 17.9)
- moved D3 74.3 mm to (18.7, 17.9)
- moved D4 74.3 mm to (65.0, 17.9)
- moved SW2 45.7 mm to (79.2, 15.4)
- moved C1 45.7 mm to (104.8, 23.7)
- moved R4 45.7 mm to (88.4, 21.3)
- moved SW3 45.7 mm to (89.3, 15.4)
- moved C2 45.7 mm to (84.4, 23.7)
- moved C3 45.7 mm to (94.6, 23.7)
- moved R2 45.7 mm to (98.6, 21.3)
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Connections:
- D3 pad 1: Net-(D2-Pad6) -> DI
- D3 pad 2: Net-(D2-Pad5) -> CI
Routing:
- net 3v3: track 30.9 -> 442.2 mm, vias 3 -> 23
- net 5v: track 6.83 -> 336.9 mm, vias 0 -> 16
- net SDA: track 0.00 -> 241.0 mm, vias 0 -> 8
- net 12v: track 13.9 -> 190.6 mm, vias 0 -> 6
- net SCL: track 0.00 -> 163.3 mm, vias 0 -> 11
- net IR: track 0.00 -> 122.8 mm, vias 0 -> 4
- net Push_1: track 2.41 -> 122.9 mm, vias 0 -> 6
- net Push_3: track 2.41 -> 108.6 mm, vias 0 -> 4
- net Push_2: track 2.39 -> 100.0 mm, vias 0 -> 6
- net DI: track 0.00 -> 71.3 mm, vias 0 -> 4
- net Net-(D4-Pad6): track 0.00 -> 65.6 mm, vias 0 -> 6
- net Net-(D4-Pad5): track 0.00 -> 65.5 mm, vias 0 -> 6
- net Net-(Q2-Pad3): track 92.8 -> 157.6 mm, vias 6 -> 9
- net CI: track 0.00 -> 58.8 mm, vias 0 -> 4
- net Net-(D5-Pad6): track 0.00 -> 45.1 mm, vias 0 -> 2
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Other:
- board text added: "3v3"
- board text added: "GND"
- board text added: "SCL"
- board text added: "SDA"

Commit message: maj schema + route
Parts:
- added D2: LED, LED_THT:LED_D3.0mm, F.Cu at (116.3, 65.0)
- added D6: LED, LED_THT:LED_D3.0mm, F.Cu at (116.3, 44.9)
- added R10: 470, Resistor_SMD:R_0805_2012Metric_Pad1.20x1.40mm_HandSolder, B.Cu at (-101.8, 22.7)
- moved R9 160.3 mm to (-109.8, 26.3)
- moved R8 156.6 mm to (-97.2, 16.1)
- moved U3 126.1 mm to (-83.9, 56.5), turned to 0 degrees
- moved J5 122.8 mm to (-70.8, 20.9)
- moved U7 40.1 mm to (134.9, 74.8), turned to 90 degrees
- moved Q1 21.6 mm to (108.5, 64.6)
- moved Q2 21.6 mm to (108.5, 44.7)
- moved D1 21.2 mm to (211.5, 91.9), turned to 180 degrees
- moved U1 18.2 mm to (211.5, 74.7)
- moved C4 18.2 mm to (212.4, 29.9)
- moved U2 12.7 mm to (208.3, 24.5), turned to 180 degrees
- moved J1 11.0 mm to (200.9, 82.9)
- moved U5 7.87 mm to (85.0, 74.8)
- moved U4 7.31 mm to (51.2, 74.8)
- moved C5 7.30 mm to (199.0, 24.5), turned to 90 degrees
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Connections:
- U4 pad 8: /a8 -> Net-(U4-Pad8)
- U7 pad 2: /b4 -> /b2
- U7 pad 3: /b7 -> /b3
- U7 pad 4: /b2 -> /b4
- U7 pad 6: /b9 -> /b6
- U7 pad 7: /b3 -> /b7
- U7 pad 9: /b6 -> /b9
- U8 pad 8: /b8 -> Net-(U8-Pad8)
Routing:
- net 5v: track 336.9 -> 22.9 mm, vias 16 -> 8
- net 3v3: track 442.2 -> 169.2 mm, vias 23 -> 13
- net SDA: track 241.0 -> 59.9 mm, vias 8 -> 4
- net 12v: track 190.6 -> 17.3 mm, vias 6 -> 0
- net Net-(D2-Pad2): track 169.0 -> 17.2 mm, vias 8 -> 2
- net Net-(D6-Pad2): track 157.6 -> 13.9 mm, vias 9 -> 2
- net SCL: track 163.3 -> 37.0 mm, vias 11 -> 3
- net IR: track 122.8 -> 4.29 mm, vias 4 -> 1
- net /b6: track 142.8 -> 41.8 mm, vias 4 -> 2
- net /b8: track 129.7 -> 34.7 mm, vias 4 -> 1
- net /a8: track 94.4 -> 0.03 mm, vias 4 -> 0
- net /b9: track 131.3 -> 38.6 mm, vias 4 -> 2
- net /a10: track 92.0 -> 0.00 mm, vias 4 -> 0
- net /a9: track 91.9 -> 0.04 mm, vias 4 -> 0
- net /a6: track 87.6 -> 0.04 mm, vias 4 -> 0
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