File: pcb/neOClock/neOClock.kicad_pcb (KiCad board)
At the start: 2 copper layers, 200 x 80 mm, 46 parts, among them J1 Barrel_Jack, J2 Conn_01x04, J3 Conn_01x04, J4 Conn_01x04, J5 ATECC508A, Q1 2n2222a, Q2 2n2222a, SW1 G71Y, SW2 G71Y, SW3 G71Y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

Commit message: update
Parts:
- added R11: 470, Resistor_SMD:R_0805_2012Metric_Pad1.20x1.40mm_HandSolder, B.Cu at (114.0, 80.1)
- R1: value 15k -> 47k
Connections:
- IR1 pad 2: IR -> Net-(IR1-Pad2)
- R1 pad 1: IR -> Net-(IR1-Pad2)
Routing:
- net Net-(IR1-Pad2): track 0.00 -> 6.76 mm, vias 0 -> 1
- net IR: track 4.29 -> 0.00 mm, vias 1 -> 0
- net Net-(D8-Pad5): track 42.1 -> 41.4 mm
- net 0: vias 10 -> 42
- net (no net): vias 0 -> 28

Commit message: update
Parts:
- moved Q2 11.1 mm to (111.2, 34.0)
- moved Q1 10.4 mm to (111.2, 74.6)
Routing:
- net 5v: track 22.9 -> 296.5 mm, vias 8 -> 17
- net 3v3: track 169.2 -> 260.5 mm, vias 13 -> 16
- net Push_1: track 107.3 -> 26.0 mm, vias 4 -> 2
- net /a8: track 0.03 -> 74.1 mm, vias 0 -> 3
- net Push_3: track 97.5 -> 26.1 mm, vias 4 -> 2
- net Push_2: track 86.9 -> 25.8 mm, vias 4 -> 2
- net /a2: track 0.04 -> 55.3 mm, vias 0 -> 3
- net /a9: track 0.04 -> 54.4 mm, vias 0 -> 3
- net /a10: track 0.00 -> 54.3 mm, vias 0 -> 3
- net /a3: track 0.04 -> 52.3 mm, vias 0 -> 3
- net /a6: track 0.04 -> 52.1 mm, vias 0 -> 3
- net /a7: track 0.00 -> 49.2 mm, vias 0 -> 3
- net /a4: track 0.00 -> 48.1 mm, vias 0 -> 3
- net /b7: track 40.2 -> 58.2 mm, vias 2 -> 3
- net /b6: track 41.8 -> 58.1 mm, vias 2 -> 3
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