File: pcb/neOClock/neOClock.sch (KiCad schematic (older format))
At the start: 8 parts, among them J2 Conn_01x04, J3 Conn_01x04, J4 Conn_01x04, SW1 SW_Push, SW2 SW_Push, SW3 SW_Push, U3 ESP32_dev_30p

Commit message: update
Parts:
- added C1, C4: 470µF, Capacitor_THT:CP_Radial_D5.0mm_P2.50mm, symbol Device:CP
- added C2: 100µF, Capacitor_Tantalum_SMD:CP_EIA-3216-18_Kemet-A_Pad1.58x1.35mm_HandSolder, symbol Device:C
- added D2, D3, D4, D5: APA102, LED_SMD:LED_RGB_5050-6, symbol LED:APA102
- added D6, D7, D?: LED, LED_THT:LED_D5.0mm, symbol Device:LED
- added J1: Barrel_Jack, Connector_BarrelJack:BarrelJack_CUI_PJ-036AH-SMT_Horizontal, symbol Connector:Barrel_Jack
- added J5: 78_01_030_0004, neosensor_addon:HARTING_78_01_030_0004, symbol 78_01_030_0004:78_01_030_0004
- added Q1: BC337, Package_TO_SOT_SMD:SC-59_Handsoldering, symbol Device:Q_NPN_CBE
- added Q2: Q_NPN_CBE, Package_TO_SOT_SMD:SC-59_Handsoldering, symbol Device:Q_NPN_CBE
- added U1: YAAJ_DCDC_StepDown_LM2596, neosensor_addon:DC_DC_LM2596, symbol DC_DC_LM2596:YAAJ_DCDC_StepDown_LM2596
- added U2: AMS1117, Package_TO_SOT_SMD:SOT-223-3_TabPin2, symbol Regulator_Linear:AMS1117
- added U4, U5, U7, U8: HDSP-7801, Display_7Segment:SBC18-11SURKCGKWA, symbol Display_Character:HDSP-7801
- added U6: SAA1064, SAA1064, symbol SAA1064:SAA1064
- SW1, SW2, SW3: footprint Button_Switch_SMD:SW_Push_1P1T_NO_CK_KMR2 -> Button_Switch_SMD:SW_Push_1P1T_NO_6x6mm_H9.5mm
Connections:
- net labels added: 12v, 3v3, 5v, CI, DI, IR, Push_1, Push_2, Push_3, SCL, SDA
- wire segments 78 -> 102
- no-connect marks 20 -> 25
Other:
- note added: "ATECC508A-SSHDA-T"
- note added: "EKMC1601112"
- moved on the sheet: IR1, J2, J3, J4, U3

Commit message: update
Parts:
- J5: footprint neosensor_addon:HARTING_78_01_030_0004 -> neosensor_addon:ATECC508A; symbol 78_01_030_0004:78_01_030_0004 -> neOClock-rescue:78_01_030_0004-78_01_030_0004
- U6: footprint SAA1064 -> neosensor_addon:SAA1064
- gave numbers to parts that had none: 1
Changed lines of the file:
@@
 F 0 "U6" H 9550 4942 50  0000 C CNN
 F 1 "SAA1064" H 9550 4851 50  0000 C CNN
-F 2 "SAA1064" H 9550 3775 50  0001 L BNN
+F 2 "neosensor_addon:SAA1064" H 9550 3775 50  0001 L BNN
 F 3 "" H 9550 3775 50  0001 L BNN
 	1    9550 3775
@@
 	7935 890  7935 1720
 $Comp
-L 78_01_030_0004:78_01_030_0004 J5
+L neOClock-rescue:78_01_030_0004-78_01_030_0004 J5
 U 1 1 6124A331
 P 2690 2130
 F 0 "J5" H 2690 2497 50  0000 C CNN
 F 1 "78_01_030_0004" H 2690 2406 50  0000 C CNN
-F 2 "neosensor_addon:HARTING_78_01_030_0004" H 2690 2130 50  0001 L BNN
+F 2 "neosensor_addon:ATECC508A" H 2690 2130 50  0001 L BNN
 F 3 "" H 2690 2130 50  0001 L BNN
 F 4 "Harting" H 2690 2130 50  0001 L BNN "MANUFACTURER"
@@
 EKMC1601112
 $Comp
-L Device:LED D?
+L Device:LED D1
 U 1 1 60BAEB43
 P 1505 6350
-F 0 "D?" H 1498 6566 50  0000 C CNN
+F 0 "D1" H 1498 6566 50  0000 C CNN
 F 1 "LED" H 1498 6475 50  0000 C CNN
 F 2 "LED_THT:LED_D5.0mm" H 1505 6350 50  0001 C CNN

Commit message: update
Parts:
- removed J5: 78_01_030_0004, neosensor_addon:ATECC508A, symbol neOClock-rescue:78_01_030_0004-78_01_030_0004
- removed SW1, SW2, SW3: SW_Push, Button_Switch_SMD:SW_Push_1P1T_NO_6x6mm_H9.5mm, symbol Switch:SW_Push
- removed U1: YAAJ_DCDC_StepDown_LM2596, neosensor_addon:DC_DC_LM2596, symbol DC_DC_LM2596:YAAJ_DCDC_StepDown_LM2596
- removed U6: SAA1064, neosensor_addon:SAA1064, symbol SAA1064:SAA1064
- added D10, D11, D12, D13, D14, D15, D8, D9: APA102, LED_SMD:LED_RGB_5050-6, symbol LED:APA102
- added H1, H2, H3, H4: MountingHole_Pad, MountingHole:MountingHole_3.2mm_M3_Pad, symbol Mechanical:MountingHole_Pad
- added J5: ATECC508A, neosensor_addon:ATECC508A, symbol neosensor_addon:ATECC508A
- added SW1, SW2, SW3: G71Y, neosensor_addon:G71Y_µsw_smd, symbol neosensor_addon:G71Y
- added U1: DCDC_LM2596, neosensor_addon:DC_DC_LM2596, symbol neosensor_addon:DCDC_LM2596
- added U6: SAA1064, SAA1064, symbol neosensor_addon:SAA1064
Connections:
- wire segments 102 -> 127
Other:
- moved on the sheet: C1, C2, C4, D1, D2, D3, D4, D5, IR1, J1, U2, U3

Commit message: mise a jour des schema
Parts:
- removed C1: 470µF, Capacitor_THT:CP_Radial_D5.0mm_P2.50mm, symbol Device:CP
- removed C2: 100µF, Capacitor_Tantalum_SMD:CP_EIA-3216-18_Kemet-A_Pad1.58x1.35mm_HandSolder, symbol Device:C
- removed D1: LED, LED_THT:LED_D5.0mm, symbol Device:LED
- removed SW2, SW3: G71Y, neosensor_addon:G71Y_µsw_smd, symbol neosensor_addon:G71Y
- added C?: 100µF, symbol Device:CP_Small
- added C? (x3): 1µF, symbol Device:C
- added C?: 100nF, symbol Device:C
- added D?: 1N4148, Diode_THT:D_DO-35_SOD27_P7.62mm_Horizontal, symbol Diode:1N4148
- added H5: MountingHole_Pad, MountingHole:MountingHole_3.2mm_M3_Pad, symbol Mechanical:MountingHole_Pad
- added R? (x6): 15K, symbol Device:R
- added R? (x2): 4.7K, symbol Device:R
- added R?: 15k, symbol Device:R
- added SW? (x2): G71Y, neosensor_addon:G71Y_µsw_smd, symbol neosensor_addon:G71Y
- J1: footprint Connector_BarrelJack:BarrelJack_CUI_PJ-036AH-SMT_Horizontal -> Connector_BarrelJack:BarrelJack_Horizontal
- J5: footprint neosensor_addon:ATECC508A -> neosensor_addon:SOIC-8_3.9x5.4mm_P1.27mm_HandSolder
- Q1: value BC337 -> 2n2222a
- Q2: value Q_NPN_CBE -> 2n2222a; footprint Package_TO_SOT_SMD:SC-59_Handsoldering -> Package_TO_SOT_THT:TO-92
- U6: footprint SAA1064 -> neosensor_addon:SOIC-24W_7.5x15.4mm_P1.27mm_HandSolder
Connections:
- wire segments 127 -> 154
- no-connect marks 25 -> 2
Other:
- note removed: "ATECC508A-SSHDA-T"
- note removed: "EKMC1601112"
- moved on the sheet: C4, D10, D11, D12, D13, D14, D15, D2, D3, D4, D5, D6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

Commit message: update
Parts:
- removed C4: 470µF, Capacitor_THT:CP_Radial_D5.0mm_P2.50mm, symbol Device:CP
- removed D6, D7: LED, LED_THT:LED_D5.0mm, symbol Device:LED
- removed H5: MountingHole_Pad, MountingHole:MountingHole_3.2mm_M3_Pad, symbol Mechanical:MountingHole_Pad
- C1, C2, C3, C4: renamed from C?; footprint (none) -> Resistor_SMD:R_0805_2012Metric_Pad1.20x1.40mm_HandSolder
- C5: renamed from C?; footprint (none) -> Capacitor_THT:CP_Radial_D5.0mm_P2.50mm
- R1, R2, R3, R4, R5, R6, R7, R8, R9: renamed from R?; footprint (none) -> Resistor_SMD:R_0805_2012Metric_Pad1.20x1.40mm_HandSolder
- gave numbers to parts that had none: 3
Connections:
- net labels added: a1, a10, a2, a3, a4, a5, a7, a8, a9, b1, b10, b2, b3, b4, b5, b7, b8, b9
- wire segments 154 -> 137
- no-connect marks 2 -> 21
Other:
- moved on the sheet: Q1, Q2, R8, R9, U3, U4, U5, U6

Commit message: update
Parts:
- removed U4, U5, U7, U8: HDSP-7801, Display_7Segment:SBC18-11SURKCGKWA, symbol Display_Character:HDSP-7801
- added U4, U5, U7, U8: SA15-11GWA, Display_7Segment:SA15-11xxx, symbol Display_Character:SA15-11GWA
- Q1: footprint Package_TO_SOT_SMD:SC-59_Handsoldering -> Package_TO_SOT_THT:TO-92
Connections:
- net a5 is gone; now on net a3: U6.7 (P4)
- net b5 is gone; now on net b3: U6.18 (P12)
- net a10: now also U6.4 (P7), U4.10 (G), U5.10 (G); no longer U6.10 (P1)
- net a2: now also U6.6 (P5), U4.2 (E), U5.2 (E); no longer U6.5 (P6)
- net a3: now also U4.3 (D), U5.3 (D); no longer U6.4 (P7)
- net a4: now also U6.8 (P3), U4.4 (C), U5.4 (C); no longer U6.6 (P5)
- net a7: now also U6.10 (P1), U4.7 (A), U5.7 (A); no longer U6.3 (P8)
- net a8: now also U6.3 (P8), U4.8 (DP), U5.8 (DP); no longer U6.8 (P3)
- net a9: now also U6.5 (P6), U4.9 (F), U5.9 (F); no longer U6.9 (P2)
- net b10: now also U6.21 (P15), U7.10 (G), U8.10 (G); no longer U6.15 (P9)
- net b2: now also U6.19 (P13), U7.4 (C), U8.2 (E); no longer U6.20 (P14)
- net b3: now also U7.7 (A), U8.3 (D); no longer U6.21 (P15)
- net b4: now also U6.17 (P11), U7.2 (E), U8.4 (C); no longer U6.19 (P13)
- net b7: now also U6.15 (P9), U7.3 (D), U8.7 (A); no longer U6.22 (P16)
- net b8: now also U6.22 (P16), U7.8 (DP), U8.8 (DP); no longer U6.17 (P11)
- net b9: now also U6.20 (P14), U7.6 (B), U8.9 (F); no longer U6.16 (P10)
- net at Q1.3 (E): now also U4.1 (CA), U4.5 (CA), U7.1 (CA), U7.5 (CA)
- net at Q2.3 (E): now also U5.1 (CA), U5.5 (CA), U8.1 (CA), U8.5 (CA)
- net a1 renamed a1_5
- net b1 renamed b1_5
- new net a6: U4.6 (B), U5.6 (B), U6.9 (P2)
- new net b6: U6.16 (P10), U7.9 (F), U8.6 (B)

Commit message: update
Parts:
- removed D10, D11, D12, D13, D14, D15, D2: APA102, LED_SMD:LED_RGB_5050-6, symbol LED:APA102
- D3, D4, D5, D8, D9: footprint LED_SMD:LED_RGB_5050-6 -> LED_SMD:LED_WS2812_PLCC6_5.0x5.0mm_P1.6mm
Connections:
- net CI: now also D3.2 (CI)
- net DI: now also D3.1 (DI)
Changed lines of the file:
@@
-$EndComp
-$Comp
-L LED:APA102 D2
-U 1 1 61274911
-P 1150 5900
-F 0 "D2" H 1150 6381 50  0000 C CNN
-F 1 "APA102" H 1150 6290 50  0000 C CNN
-F 2 "LED_SMD:LED_RGB_5050-6" H 1200 5600 50  0001 L TNN
-F 3 "http://www.led-color.com/upload/201506/APA102%20LED.pdf" H 1250 5525 50  0001 L TNN
-	1    1150 5900
-	1    0    0    -1
 $EndComp
 $Comp
@@
 F 0 "D3" H 1750 6381 50  0000 C CNN
 F 1 "APA102" H 1750 6290 50  0000 C CNN
-F 2 "LED_SMD:LED_RGB_5050-6" H 1800 5600 50  0001 L TNN
+F 2 "LED_SMD:LED_WS2812_PLCC6_5.0x5.0mm_P1.6mm" H 1800 5600 50  0001 L TNN
 F 3 "http://www.led-color.com/upload/201506/APA102%20LED.pdf" H 1850 5525 50  0001 L TNN
 	1    1750 5900
@@
 F 0 "D4" H 2350 6381 50  0000 C CNN
 F 1 "APA102" H 2350 6290 50  0000 C CNN
-F 2 "LED_SMD:LED_RGB_5050-6" H 2400 5600 50  0001 L TNN
+F 2 "LED_SMD:LED_WS2812_PLCC6_5.0x5.0mm_P1.6mm" H 2400 5600 50  0001 L TNN
 F 3 "http://www.led-color.com/upload/201506/APA102%20LED.pdf" H 2450 5525 50  0001 L TNN
 	1    2350 5900
@@
 F 0 "D5" H 2950 6381 50  0000 C CNN
 F 1 "APA102" H 2950 6290 50  0000 C CNN
-F 2 "LED_SMD:LED_RGB_5050-6" H 3000 5600 50  0001 L TNN
+F 2 "LED_SMD:LED_WS2812_PLCC6_5.0x5.0mm_P1.6mm" H 3000 5600 50  0001 L TNN
 F 3 "http://www.led-color.com/upload/201506/APA102%20LED.pdf" H 3050 5525 50  0001 L TNN
 	1    2950 5900
@@
 Text GLabel 850  5600 0    50   Input ~ 0
 5v
-Text GLabel 850  5800 0    50   Input ~ 0
-DI
-Text GLabel 850  5900 0    50   Input ~ 0
-CI
 $Comp
 L neosensor_addon:ATECC508A J5
@@
 F 0 "D8" H 3550 6381 50  0000 C CNN
 F 1 "APA102" H 3550 6290 50  0000 C CNN
-F 2 "LED_SMD:LED_RGB_5050-6" H 3600 5600 50  0001 L TNN
+F 2 "LED_SMD:LED_WS2812_PLCC6_5.0x5.0mm_P1.6mm" H 3600 5600 50  0001 L TNN
 F 3 "http://www.led-color.com/upload/201506/APA102%20LED.pdf" H 3650 5525 50  0001 L TNN
 	1    3550 5900
@@
 F 0 "D9" H 4150 6381 50  0000 C CNN
 F 1 "APA102" H 4150 6290 50  0000 C CNN
-F 2 "LED_SMD:LED_RGB_5050-6" H 4200 5600 50  0001 L TNN
+F 2 "LED_SMD:LED_WS2812_PLCC6_5.0x5.0mm_P1.6mm" H 4200 5600 50  0001 L TNN
 F 3 "http://www.led-color.com/upload/201506/APA102%20LED.pdf" H 4250 5525 50  0001 L TNN
 	1    4150 5900
-	1    0    0    -1
-$EndComp
-$Comp
-L LED:APA102 D10
-U 1 1 60B65103
-P 4750 5900
-F 0 "D10" H 4750 6381 50  0000 C CNN
-F 1 "APA102" H 4750 6290 50  0000 C CNN
-F 2 "LED_SMD:LED_RGB_5050-6" H 4800 5600 50  0001 L TNN
-F 3 "http://www.led-color.com/upload/201506/APA102%20LED.pdf" H 4850 5525 50  0001 L TNN
-	1    4750 5900
-	1    0    0    -1
-$EndComp
-$Comp
-L LED:APA102 D11
-U 1 1 60B65109
-P 5350 5900
-F 0 "D11" H 5350 6381 50  0000 C CNN
-F 1 "APA102" H 5350 6290 50  0000 C CNN
-F 2 "LED_SMD:LED_RGB_5050-6" H 5400 5600 50  0001 L TNN
-F 3 "http://www.led-color.com/upload/201506/APA102%20LED.pdf" H 5450 5525 50  0001 L TNN
-	1    5350 5900
-	1    0    0    -1
-$EndComp
-$Comp
-L LED:APA102 D12
-U 1 1 60B6B69E
-P 5950 5900
-F 0 "D12" H 5950 6381 50  0000 C CNN
-F 1 "APA102" H 5950 6290 50  0000 C CNN
-F 2 "LED_SMD:LED_RGB_5050-6" H 6000 5600 50  0001 L TNN
-F 3 "http://www.led-color.com/upload/201506/APA102%20LED.pdf" H 6050 5525 50  0001 L TNN
-	1    5950 5900
-	1    0    0    -1
-$EndComp
-$Comp
-L LED:APA102 D13
-U 1 1 60B6B6A4
-P 6550 5900
-F 0 "D13" H 6550 6381 50  0000 C CNN
-F 1 "APA102" H 6550 6290 50  0000 C CNN
-F 2 "LED_SMD:LED_RGB_5050-6" H 6600 5600 50  0001 L TNN
-F 3 "http://www.led-color.com/upload/201506/APA102%20LED.pdf" H 6650 5525 50  0001 L TNN
-	1    6550 5900
-	1    0    0    -1
-$EndComp
-$Comp
-L LED:APA102 D14
-U 1 1 60B6B6AA
-P 7150 5900
-F 0 "D14" H 7150 6381 50  0000 C CNN
-F 1 "APA102" H 7150 6290 50  0000 C CNN
-F 2 "LED_SMD:LED_RGB_5050-6" H 7200 5600 50  0001 L TNN
-F 3 "http://www.led-color.com/upload/201506/APA102%20LED.pdf" H 7250 5525 50  0001 L TNN
-	1    7150 5900
-	1    0    0    -1
-$EndComp
-$Comp
-L LED:APA102 D15
-U 1 1 60B6B6B0
-P 7750 5900
-F 0 "D15" H 7750 6381 50  0000 C CNN
-F 1 "APA102" H 7750 6290 50  0000 C CNN
-F 2 "LED_SMD:LED_RGB_5050-6" H 7800 5600 50  0001 L TNN
-F 3 "http://www.led-color.com/upload/201506/APA102%20LED.pdf" H 7850 5525 50  0001 L TNN
-	1    7750 5900
 	1    0    0    -1
 $EndComp
@@
 Text GLabel 750  2350 0    50   Input ~ 0
 3v3
-NoConn ~ 8050 5800
-NoConn ~ 8050 5900
-Wire Wire Line
-	850  5600 1150 5600
-Connection ~ 1150 5600
-Wire Wire Line
-	1150 5600 1750 5600
+NoConn ~ 4450 5800
+NoConn ~ 4450 5900
 Connection ~ 1750 5600
 Wire Wire Line
@@
 Wire Wire Line
 	3550 5600 4150 5600
-Connection ~ 4150 5600
-Wire Wire Line
-	4150 5600 4750 5600
-Connection ~ 4750 5600
-Wire Wire Line
-	4750 5600 5350 5600
-Connection ~ 5350 5600
-Wire Wire Line
-	5350 5600 5950 5600
-Connection ~ 5950 5600
-Wire Wire Line
-	5950 5600 6550 5600
-Connection ~ 6550 5600
-Wire Wire Line
-	6550 5600 7150 5600
-Connection ~ 7150 5600
-Wire Wire Line
-	7150 5600 7750 5600
-Wire Wire Line
-	850  6200 1150 6200
-Connection ~ 1150 6200
-Wire Wire Line
-	1150 6200 1750 6200
 Connection ~ 1750 6200
 Wire Wire Line
@@
 Wire Wire Line
 	3550 6200 4150 6200
-Connection ~ 4150 6200
-Wire Wire Line
-	4150 6200 4750 6200
-Connection ~ 4750 6200
-Wire Wire Line
-	4750 6200 5350 6200
-Connection ~ 5350 6200
-Wire Wire Line
-	5350 6200 5950 6200
-Connection ~ 5950 6200
-Wire Wire Line
-	5950 6200 6550 6200
-Connection ~ 6550 6200
-Wire Wire Line
-	6550 6200 7150 6200
-Connection ~ 7150 6200
-Wire Wire Line
-	7150 6200 7750 6200
 $Comp
 L pspice:0 #GND0114
@@
 Wire Wire Line
 	9150 1100 9150 1000
+Connection ~ 9150 1000
+Wire Wire Line
+	850  6200 1750 6200
+Wire Wire Line
+	850  5600 1750 5600
+Text GLabel 850  5900 0    50   Input ~ 0
+CI
+Text GLabel 850  5800 0    50   Input ~ 0
+DI
+Wire Wire Line
+	850  5800 1450 5800
+Wire Wire Line
+	850  5900 1450 5900
 Wire Bus Line
 	9950 1100 9950 2950
 Wire Bus Line
 	8325 1100 8325 2950
-Connection ~ 9150 1000
 $EndSCHEMATC

Commit message: maj schema + route
Parts:
- added D2, D6: LED, LED_THT:LED_D3.0mm, symbol Device:LED
- added R10: 470, Resistor_SMD:R_0805_2012Metric_Pad1.20x1.40mm_HandSolder, symbol Device:R
Connections:
- net a8: now also D2.1 (K); no longer U4.8 (DP)
- net b2: now also U7.2 (E); no longer U7.4 (C)
- net b3: now also U7.3 (D); no longer U7.7 (A)
- net b4: now also U7.4 (C); no longer U7.2 (E)
- net b6: now also U7.6 (B); no longer U7.9 (F)
- net b7: now also U7.7 (A); no longer U7.3 (D)
- net b8: now also D6.1 (K); no longer U8.8 (DP)
- net b9: now also U7.9 (F); no longer U7.6 (B)
- net at U3.13 (GPIO1): now also R10.2
- net at Q1.3 (E), U4.1 (CA), U4.5 (CA)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: now also D2.2 (A)
- net at Q2.3 (E), U5.1 (CA), U5.5 (CA)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: now also D6.2 (A)
- no-connect marks 21 -> 23
Other:
- moved on the sheet: U7
Changed lines of the file:
@@
 Text Label 8125 1500 0    50   ~ 0
 a9
-Text Label 8125 1700 0    50   ~ 0
+Text Label 7225 1500 2    50   ~ 0
 a8
 Text Label 8125 1100 0    50   ~ 0
@@
 Wire Wire Line
 	8125 1600 8225 1600
-Wire Wire Line
-	8125 1700 8225 1700
 Entry Wire Line
 	8225 1000 8325 1100
@@
 Entry Wire Line
 	8225 1600 8325 1700
-Entry Wire Line
-	8225 1700 8325 1800
 Text Label 8525 1600 2    50   ~ 0
 a10
@@
 b7
 Entry Wire Line
-	10050 1700 9950 1800
-Entry Wire Line
 	10050 1600 9950 1700
 Entry Wire Line
@@
 Entry Wire Line
 	10050 1000 9950 1100
-Wire Wire Line
-	10150 1700 10050 1700
 Wire Wire Line
 	10150 1600 10050 1600
@@
 Text Label 10150 1100 2    50   ~ 0
 b6
-Text Label 10150 1700 2    50   ~ 0
+Text Label 11050 1500 0    50   ~ 0
 b8
 Text Label 10150 1500 2    50   ~ 0
@@
 Wire Wire Line
 	9750 1000 9850 1000
+Text Label 9750 1000 0    50   ~ 0
+b7
+Text Label 9750 1300 0    50   ~ 0
+b3
 Text Label 9750 1400 0    50   ~ 0
-b7
+b2
+Text Label 9750 1200 0    50   ~ 0
+b4
+Text Label 9750 1100 0    50   ~ 0
+b6
 Text Label 9750 1700 0    50   ~ 0
-b3
+b8
 Text Label 9750 1500 0    50   ~ 0
-b2
-Text Label 9750 1300 0    50   ~ 0
-b4
-Text Label 9750 1200 0    50   ~ 0
-b6
-Text Label 9750 1000 0    50   ~ 0
-b8
+b9
 Text Label 9750 1600 0    50   ~ 0
-b9
-Text Label 9750 1100 0    50   ~ 0
 b10
 $Comp
@@
 NoConn ~ 6500 3900
 NoConn ~ 6500 3700
-NoConn ~ 6500 3600
+NoConn ~ 6850 3600
 $Comp
 L Display_Character:SA15-11GWA U4
@@
 	9125 1600 9125 1700
 Wire Wire Line
-	7525 600  7525 1600
+	7525 600  7525 1500
 Wire Wire Line
 	7525 1700 7525 1725
@@
 Connection ~ 7525 1600
 Connection ~ 7525 1700
-Wire Wire Line
-	10750 575  10750 1600
 $Comp
 L Display_Character:SA15-11GWA U8
@@
 L Display_Character:SA15-11GWA U7
 U 1 1 60C42FF4
-P 9450 1400
-F 0 "U7" H 9450 733 50  0000 C CNN
-F 1 "SA15-11GWA" H 9450 824 50  0000 C CNN
-F 2 "Display_7Segment:SA15-11xxx" H 9450 1350 50  0001 C CNN
-F 3 "http://www.kingbrightusa.com/images/catalog/SPEC/SA15-11GWA.pdf" H 9450 1350 50  0001 C CNN
-	1    9450 1400
-	-1   0    0    1
-$EndComp
-Wire Wire Line
-	9150 600  9150 1000
-Wire Wire Line
-	9150 1100 9150 1000
-Connection ~ 9150 1000
+P 9450 1300
+F 0 "U7" H 9450 633 50  0000 C CNN
+F 1 "SA15-11GWA" H 9450 724 50  0000 C CNN
+F 2 "Display_7Segment:SA15-11xxx" H 9450 1250 50  0001 C CNN
+F 3 "http://www.kingbrightusa.com/images/catalog/SPEC/SA15-11GWA.pdf" H 9450 1250 50  0001 C CNN
+	1    9450 1300
+	-1   0    0    -1
+$EndComp
 Wire Wire Line
 	850  6200 1750 6200
@@
 Wire Wire Line
 	850  5900 1450 5900
+Wire Wire Line
+	6500 3600 6550 3600
+$Comp
+L Device:R R10
+U 1 1 60C86E5A
+P 6700 3600
+F 0 "R10" V 6800 3525 50  0000 C CNN
+F 1 "470" V 6800 3725 50  0000 C CNN
+F 2 "Resistor_SMD:R_0805_2012Metric_Pad1.20x1.40mm_HandSolder" V 6630 3600 50  0001 C CNN
+F 3 "~" H 6700 3600 50  0001 C CNN
+	1    6700 3600
+	0    1    1    0
+$EndComp
+Wire Wire Line
+	9150 600  9150 1600
+Connection ~ 9150 1600
+Wire Wire Line
+	9150 1600 9150 1700
+$Comp
+L Device:LED D6
+U 1 1 60CB96E0
+P 10900 1500
+F 0 "D6" H 10893 1245 50  0000 C CNN
+F 1 "LED" H 10893 1336 50  0000 C CNN
+F 2 "LED_THT:LED_D3.0mm" H 10900 1500 50  0001 C CNN
+F 3 "~" H 10900 1500 50  0001 C CNN
+	1    10900 1500
+	-1   0    0    1
+$EndComp
+$Comp
+L Device:LED D2
+U 1 1 60CBAB59
+P 7375 1500
+F 0 "D2" H 7368 1716 50  0000 C CNN
+F 1 "LED" H 7368 1625 50  0000 C CNN
+F 2 "LED_THT:LED_D3.0mm" H 7375 1500 50  0001 C CNN
+F 3 "~" H 7375 1500 50  0001 C CNN
+	1    7375 1500
+	1    0    0    -1
+$EndComp
+Connection ~ 10750 1500
+Wire Wire Line
+	10750 1500 10750 1600
+Connection ~ 7525 1500
+Wire Wire Line
+	7525 1500 7525 1600
+Wire Wire Line
+	10750 575  10750 1500
+NoConn ~ 8125 1700
+NoConn ~ 10150 1700
 Wire Bus Line
 	9950 1100 9950 2950
