File: pcb/pcb-v5b/pcb-v5b.kicad_sch (KiCad schematic)
At the start: 48 parts, among them J1 Conn_01x04, J2 Conn_01x04, J3 Conn_01x05, J4 Conn_01x05, J5 Conn_01x05, J6 Conn_01x06, Q1 2N7002, SW1 clear, SW2 +, SW3 -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

Commit message: updated neOSensor V5B schematic
Parts:
- removed J4: Conn_01x05, Connector_PinHeader_2.54mm:PinHeader_1x05_P2.54mm_Vertical, symbol Connector_Generic:Conn_01x05
- added J4: Conn_01x07, Connector_PinHeader_2.54mm:PinHeader_1x07_P2.54mm_Vertical, symbol Connector_Generic:Conn_01x07
- added U6: ATECC608A-SSHDA, Package_SO:SOIC-8_3.9x4.9mm_P1.27mm, symbol Security:ATECC608A-SSHDA
- C1, C3, C4, C5: footprint Resistor_SMD:R_0805_2012Metric_Pad1.20x1.40mm_HandSolder -> Capacitor_SMD:C_0805_2012Metric_Pad1.18x1.45mm_HandSolder
- C2: symbol Device:CP1_Small -> Device:C_Polarized_Small_US
- C6: footprint (none) -> Capacitor_SMD:C_0805_2012Metric_Pad1.18x1.45mm_HandSolder
- D1: symbol Device:LED_Small_ALT -> Device:LED_Small_Filled
Connections:
- net +3V3: now also J4.3 (Pin_3), U6.8 (VCC)
- net GND: now also J4.4 (Pin_4), U6.4 (GND)
- net INT: now also J4.7 (Pin_7)
- net SCL: now also J4.2 (Pin_2), J4.5 (Pin_5), U6.6 (SCL)
- net SDA: now also J4.1 (Pin_1), J4.6 (Pin_6), U6.5 (SDA)
Other:
- note added: "Crypto"
- note added: "HC-SR01 V+ accepts from 5 to 20v OUT pin is 3.3 TTL"
- note added: "PWR flags (for ERC)"
- note added: "no PWR flag needed for 3v3 because the voltage regulator is a source"
- note removed: "HC-SR01 V+ accepts from 5 to 20v OUT pin is 3.3 TTL >> Remove R9 if IR sensor present <<"
- moved on the sheet: C1, C2, H1, H2, U4
